File: JetsonCarrierBoard/sodimm1.kicad_sch (KiCad schematic)
At the start: 1 part

Commit message: Files Autosaved, etc.
Connections:
- net GND: now reaches J?.1 (GND)
- net GND: now also J?.102 (GND), J?.107 (GND), J?.113 (GND), J?.119 (GND), J?.125 (GND), J?.129 (GND), J?.13 (GND), J?.132 (GND), J?.135 (GND), J?.138 (GND), J?.14 (GND), J?.141 (GND), J?.144 (GND), J?.146 (GND), J?.147 (GND), J?.152 (GND), J?.153 (GND), J?.158 (GND), J?.159 (GND), J?.164 (GND), J?.165 (GND), J?.170 (GND), J?.171 (GND), J?.176 (GND), J?.177 (GND), J?.19 (GND), J?.2 (GND), J?.20 (GND), J?.200 (GND), J?.201 (GND), J?.217 (GND), J?.231 (GND), J?.241 (GND), J?.242 (GND), J?.243 (GND), J?.244 (GND), J?.245 (GND), J?.246 (GND), J?.247 (GND), J?.248 (GND), J?.249 (GND), J?.25 (GND), J?.250 (GND), J?.26 (GND), J?.261 (GND), J?.262 (GND), J?.31 (GND), J?.32 (GND), J?.37 (GND), J?.38 (GND), J?.43 (GND), J?.44 (GND), J?.49 (GND), J?.50 (GND), J?.55 (GND), J?.56 (GND), J?.61 (GND), J?.62 (GND), J?.67 (GND), J?.68 (GND), J?.7 (GND), J?.73 (GND), J?.74 (GND), J?.79 (GND), J?.8 (GND), J?.80 (GND), J?.85 (GND), J?.86 (GND)
- net +5V: now reaches J?.251 (VDD_IN)
- net +5V: now also J?.252 (VDD_IN), J?.253 (VDD_IN), J?.254 (VDD_IN), J?.255 (VDD_IN), J?.256 (VDD_IN), J?.257 (VDD_IN), J?.258 (VDD_IN), J?.259 (VDD_IN), J?.260 (VDD_IN)
- no-connect marks 0 -> 2
