File: JetsonCarrierBoard/sodimm3.kicad_sch (KiCad schematic)
At the start: 3 parts

Commit message: Adding more Title block info and changing main hierarchical page layout
Other:
- title: (none) -> SODIMM Connector 3/3
Changed lines of the file:
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@@
 (kicad_sch (version 20211123) (generator eeschema)
   (paper "A4")
+  (title_block
+    (title "SODIMM Connector 3/3")
+    (date "2022-09-18")
+    (rev "1.0")
+  )
   (junction (at 93.98 165.1) (diameter 0) (color 0 0 0 0)
   )

Commit message: Readability improvements mostly
Other:
- note added: "DP Con"
- note added: "M.2 Key E WiFi/BT"
- note added: "NVME SSD"
- note added: "USB Type-C Con (USBSS)"
Changed lines of the file:
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@@
   (no_connect (at 96.52 73.66))
   (no_connect (at 96.52 128.27))
+  (polyline (pts (xy 187.96 147.955) (xy 189.23 147.955))
+    (stroke (width 0) (type solid) (color 0 0 0 1))
+  )
   (wire (pts (xy 165.1 113.03) (xy 172.72 113.03))
     (stroke (width 0) (type default) (color 0 0 0 0))
@@
     (stroke (width 0) (type default) (color 0 0 0 0))
   )
+  (polyline (pts (xy 187.96 122.555) (xy 189.23 122.555))
+    (stroke (width 0) (type solid) (color 0 0 0 1))
+  )
   (wire (pts (xy 96.52 146.05) (xy 69.85 146.05))
     (stroke (width 0) (type default) (color 0 0 0 0))
@@
     (stroke (width 0) (type default) (color 0 0 0 0))
   )
+  (polyline (pts (xy 77.47 127.635) (xy 78.74 127.635))
+    (stroke (width 0) (type solid) (color 0 0 0 1))
+  )
+  (polyline (pts (xy 189.23 122.555) (xy 189.23 147.955))
+    (stroke (width 0) (type solid) (color 0 0 0 1))
+  )
   (wire (pts (xy 165.1 101.6) (xy 172.72 101.6))
     (stroke (width 0) (type default) (color 0 0 0 0))
   )
+  (polyline (pts (xy 189.865 116.84) (xy 191.135 116.84))
+    (stroke (width 0) (type solid) (color 0 0 0 1))
+  )
   (wire (pts (xy 165.1 69.85) (xy 172.72 69.85))
     (stroke (width 0) (type default) (color 0 0 0 0))
@@
     (stroke (width 0) (type default) (color 0 0 0 0))
   )
+  (polyline (pts (xy 77.47 95.885) (xy 77.47 127.635))
+    (stroke (width 0) (type solid) (color 0 0 0 1))
+  )
   (wire (pts (xy 165.1 146.05) (xy 172.72 146.05))
     (stroke (width 0) (type default) (color 0 0 0 0))
@@
     (stroke (width 0) (type default) (color 0 0 0 0))
   )
+  (polyline (pts (xy 189.865 111.125) (xy 189.865 122.555))
+    (stroke (width 0) (type solid) (color 0 0 0 1))
+  )
   (wire (pts (xy 165.1 138.43) (xy 172.72 138.43))
     (stroke (width 0) (type default) (color 0 0 0 0))
@@
     (stroke (width 0) (type default) (color 0 0 0 0))
   )
+  (polyline (pts (xy 76.2 111.125) (xy 77.47 111.125))
+    (stroke (width 0) (type solid) (color 0 0 0 1))
+  )
   (wire (pts (xy 92.71 105.41) (xy 96.52 105.41))
     (stroke (width 0) (type default) (color 0 0 0 0))
   )
+  (polyline (pts (xy 189.865 122.555) (xy 188.595 122.555))
+    (stroke (width 0) (type solid) (color 0 0 0 1))
+  )
   (wire (pts (xy 165.1 140.97) (xy 172.72 140.97))
     (stroke (width 0) (type default) (color 0 0 0 0))
@@
     (stroke (width 0) (type default) (color 0 0 0 0))
   )
+  (polyline (pts (xy 189.865 47.625) (xy 189.865 111.125))
+    (stroke (width 0) (type solid) (color 0 0 0 1))
+  )
   (wire (pts (xy 165.1 49.53) (xy 172.72 49.53))
     (stroke (width 0) (type default) (color 0 0 0 0))
@@
     (stroke (width 0) (type default) (color 0 0 0 0))
   )
+  (polyline (pts (xy 188.595 47.625) (xy 189.865 47.625))
+    (stroke (width 0) (type solid) (color 0 0 0 1))
+  )
   (wire (pts (xy 165.1 63.5) (xy 172.72 63.5))
     (stroke (width 0) (type default) (color 0 0 0 0))
@@
     (stroke (width 0) (type default) (color 0 0 0 0))
   )
+  (polyline (pts (xy 189.865 78.74) (xy 191.135 78.74))
+    (stroke (width 0) (type solid) (color 0 0 0 1))
+  )
   (wire (pts (xy 165.1 109.22) (xy 172.72 109.22))
     (stroke (width 0) (type default) (color 0 0 0 0))
@@
     (stroke (width 0) (type default) (color 0 0 0 0))
   )
+  (polyline (pts (xy 189.23 134.62) (xy 190.5 134.62))
+    (stroke (width 0) (type solid) (color 0 0 0 1))
+  )
   (wire (pts (xy 165.1 83.82) (xy 172.72 83.82))
     (stroke (width 0) (type default) (color 0 0 0 0))
@@
     (stroke (width 0) (type default) (color 0 0 0 0))
   )
+  (polyline (pts (xy 78.74 95.885) (xy 77.47 95.885))
+    (stroke (width 0) (type solid) (color 0 0 0 1))
+  )
   (wire (pts (xy 165.1 115.57) (xy 172.72 115.57))
     (stroke (width 0) (type default) (color 0 0 0 0))
@@
     (stroke (width 0) (type default) (color 0 0 0 0))
   )
+  (polyline (pts (xy 188.595 111.125) (xy 189.865 111.125))
+    (stroke (width 0) (type solid) (color 0 0 0 1))
+  )
   (wire (pts (xy 165.1 97.79) (xy 172.72 97.79))
     (stroke (width 0) (type default) (color 0 0 0 0))
@@
     (stroke (width 0) (type default) (color 0 0 0 0))
   )
+  (text "DP Con" (at 75.565 111.76 180)
+    (effects (font (size 1.27 1.27)) (justify right bottom))
+  )
+  (text "USB Type-C Con (USBSS)" (at 191.77 117.475 0)
+    (effects (font (size 1.27 1.27)) (justify left bottom))
+  )
+  (text "NVME SSD" (at 191.77 80.01 0)
+    (effects (font (size 1.27 1.27)) (justify left bottom))
+  )
+  (text "M.2 Key E WiFi/BT" (at 191.135 135.255 0)
+    (effects (font (size 1.27 1.27)) (justify left bottom))
+  )
   (global_label "M2E_SUSCLK_32KHZ" (shape output) (at 101.6 165.1 0) (fields_autoplaced)
