File: JetsonCarrierBoard/imu.kicad_sch (KiCad schematic)
At the start: 0 parts

Commit message: IMU wiring
Parts:
- added C?: 0.47u, symbol Device:C
- added C?: 10n, symbol Device:C
- added C?: 0.1u, symbol Device:C
- added C?: 2.2u, symbol Device:C
- added U?: ICM-20602, Package_LGA:LGA-16_3x3mm_P0.5mm_LayoutBorder3x5y, symbol Sensor_Motion:ICM-20602
Connections:
- new net: C?.1, U?.14 (REGOUT)
- new net: C?.1, U?.1 (VDDIO)
- new net +1V8: C?.1, C?.1, U?.16 (VDD)
- new net GND: C?.2, C?.2, C?.2, C?.2, U?.10 (GND), U?.11 (GND), U?.12 (GND), U?.13 (GND), U?.15 (GND), U?.8 (FSYNC), U?.9 (GND)
- new net SPI0_CS0: U?.5 (~{CS})
- new net SPI0_MISO: U?.4 (SAO/SD0)
- new net SPI0_MOSI: U?.3 (SDA/SDI)
- new net SPI0_SCK: U?.2 (SCL/SPC)
- no-connect marks 0 -> 1

Commit message: Adding more Title block info and changing main hierarchical page layout
Other:
- title: (none) -> Inertial Measurement Unit (IMU)
Changed lines of the file:
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@@
 (kicad_sch (version 20211123) (generator eeschema)
   (paper "A4")
+  (title_block
+    (title "Inertial Measurement Unit (IMU)")
+    (date "2022-09-18")
+    (rev "1.0")
+  )
   (junction (at 132.08 90.17) (diameter 0) (color 0 0 0 0)
   )
