File: JetsonCarrierBoard/microphone.kicad_sch (KiCad schematic)
At the start: 5 parts

Commit message: Adding more Title block info and changing main hierarchical page layout
Other:
- title: (none) -> Stereo Microphone
Changed lines of the file:
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@@
 (kicad_sch (version 20211123) (generator eeschema)
   (paper "A4")
+  (title_block
+    (title "Stereo Microphone")
+    (date "2022-09-18")
+    (rev "1.0")
+  )
   (junction (at 142.24 102.87) (diameter 0) (color 0 0 0 0)
   )
