File: JetsonCarrierBoard/usbC.kicad_sch (KiCad schematic)
At the start: 23 parts

Commit message: Adding more Title block info and changing main hierarchical page layout
Other:
- title: (none) -> USB-C w/ Alt Mode DP
Changed lines of the file:
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@@
 (kicad_sch (version 20211123) (generator eeschema)
   (paper "A4")
+  (title_block
+    (title "USB-C w/ Alt Mode DP")
+    (date "2022-09-18")
+    (rev "1.0")
+  )
   (junction (at 110.49 85.09) (diameter 0) (color 0 0 0 0)
   )
