File: JetsonCarrierBoard/csi-DESKTOP-4N3HF78.kicad_sch (KiCad schematic)
At the start: 31 parts, among them U10 TS3USB30E, U11 SFW15R-1STAE1LF, U12 SFW15R-1STAE1LF

Commit message: A ton
Parts:
- renumbered C57 to C?, C56 to C?, D16 to D?, D4 to D?, D7 to D?, D11 to D?, D20 to D?, D22 to D?, D13 to D?, D21 to D?, D8 to D?, D17 to D?, D5 to D?, D9 to D?, D15 to D?, D18 to D?, D10 to D?, D6 to D?, D23 to D?, D14 to D?, D12 to D?, D19 to D?, R35 to R?, R37 to R?, R40 to R?, R39 to R?, R36 to R?, R38 to R?, U10 to U?, U12 to U?, U11 to U?
