File: JetsonCarrierBoard/dc_jack-DESKTOP-4N3HF78.kicad_sch (KiCad schematic)
At the start: 9 parts, among them J7 Barrel_Jack_MountingPin, Q10 AON6411

Commit message: A ton
Parts:
- renumbered C85 to C?, C84 to C?, C82 to C?, C83 to C?, D28 to D?, J7 to J?, Q10 to Q?, R76 to R?, R77 to R?
Changed lines of the file:
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@@
   (symbol (lib_id "Device:C") (at 199.39 97.79 0) (unit 1)
     (in_bom yes) (on_board yes) (fields_autoplaced)
-    (property "Reference" "C85" (id 0) (at 203.2 96.5199 0)
+    (property "Reference" "C?" (id 0) (at 203.2 96.5199 0)
       (effects (font (size 1.27 1.27)) (justify left))
     )
@@
   (symbol (lib_id "Device:C") (at 187.96 97.79 0) (unit 1)
     (in_bom yes) (on_board yes) (fields_autoplaced)
-    (property "Reference" "C84" (id 0) (at 191.77 96.5199 0)
+    (property "Reference" "C?" (id 0) (at 191.77 96.5199 0)
       (effects (font (size 1.27 1.27)) (justify left))
     )
@@
   (symbol (lib_id "Device:C") (at 138.43 97.79 0) (unit 1)
     (in_bom yes) (on_board yes) (fields_autoplaced)
-    (property "Reference" "C82" (id 0) (at 142.24 96.5199 0)
+    (property "Reference" "C?" (id 0) (at 142.24 96.5199 0)
       (effects (font (size 1.27 1.27)) (justify left))
     )
@@
   (symbol (lib_id "Transistor_FET:AON6411") (at 176.53 96.52 270) (mirror x) (unit 1)
     (in_bom yes) (on_board yes) (fields_autoplaced)
-    (property "Reference" "Q10" (id 0) (at 176.53 86.36 90))
+    (property "Reference" "Q?" (id 0) (at 176.53 86.36 90))
     (property "Value" "AON6411" (id 1) (at 176.53 88.9 90))
     (property "Footprint" "Package_DFN_QFN:AO_DFN-8-1EP_5.55x5.2mm_P1.27mm_EP4.12x4.6mm" (id 2) (at 174.625 91.44 0)
@@
   (symbol (lib_id "Connector:Barrel_Jack_MountingPin") (at 107.95 96.52 0) (unit 1)
     (in_bom yes) (on_board yes) (fields_autoplaced)
-    (property "Reference" "J7" (id 0) (at 107.95 87.63 0))
+    (property "Reference" "J?" (id 0) (at 107.95 87.63 0))
     (property "Value" "Barrel_Jack_MountingPin" (id 1) (at 107.95 90.17 0))
     (property "Footprint" "" (id 2) (at 109.22 97.536 0)
@@
   (symbol (lib_id "Device:R") (at 149.86 97.79 0) (unit 1)
     (in_bom yes) (on_board yes) (fields_autoplaced)
-    (property "Reference" "R76" (id 0) (at 152.4 96.5199 0)
+    (property "Reference" "R?" (id 0) (at 152.4 96.5199 0)
       (effects (font (size 1.27 1.27)) (justify left))
     )
@@
   (symbol (lib_id "Device:D_Zener") (at 123.19 97.79 270) (unit 1)
     (in_bom yes) (on_board yes) (fields_autoplaced)
-    (property "Reference" "D28" (id 0) (at 125.73 96.5199 90)
+    (property "Reference" "D?" (id 0) (at 125.73 96.5199 90)
       (effects (font (size 1.27 1.27)) (justify left))
     )
@@
   (symbol (lib_id "power:GND") (at 187.96 104.14 0) (unit 1)
     (in_bom yes) (on_board yes) (fields_autoplaced)
-    (property "Reference" "#PWR0187" (id 0) (at 187.96 110.49 0)
+    (property "Reference" "#PWR?" (id 0) (at 187.96 110.49 0)
       (effects (font (size 1.27 1.27)) hide)
     )
@@
   (symbol (lib_id "power:GND") (at 138.43 104.14 0) (unit 1)
     (in_bom yes) (on_board yes) (fields_autoplaced)
-    (property "Reference" "#PWR0185" (id 0) (at 138.43 110.49 0)
+    (property "Reference" "#PWR?" (id 0) (at 138.43 110.49 0)
       (effects (font (size 1.27 1.27)) hide)
     )
@@
   (symbol (lib_id "power:GND") (at 123.19 104.14 0) (unit 1)
     (in_bom yes) (on_board yes) (fields_autoplaced)
-    (property "Reference" "#PWR0184" (id 0) (at 123.19 110.49 0)
+    (property "Reference" "#PWR?" (id 0) (at 123.19 110.49 0)
       (effects (font (size 1.27 1.27)) hide)
     )
@@
   (symbol (lib_id "power:+BATT") (at 199.39 91.44 0) (unit 1)
     (in_bom yes) (on_board yes) (fields_autoplaced)
-    (property "Reference" "#PWR0188" (id 0) (at 199.39 95.25 0)
+    (property "Reference" "#PWR?" (id 0) (at 199.39 95.25 0)
       (effects (font (size 1.27 1.27)) hide)
     )
@@
   (symbol (lib_id "power:GND") (at 199.39 104.14 0) (unit 1)
     (in_bom yes) (on_board yes) (fields_autoplaced)
-    (property "Reference" "#PWR0189" (id 0) (at 199.39 110.49 0)
+    (property "Reference" "#PWR?" (id 0) (at 199.39 110.49 0)
       (effects (font (size 1.27 1.27)) hide)
     )
@@
   (symbol (lib_id "Device:C") (at 162.56 97.79 0) (unit 1)
     (in_bom yes) (on_board yes) (fields_autoplaced)
-    (property "Reference" "C83" (id 0) (at 166.37 96.5199 0)
+    (property "Reference" "C?" (id 0) (at 166.37 96.5199 0)
       (effects (font (size 1.27 1.27)) (justify left))
     )
@@
   (symbol (lib_id "power:GND") (at 115.57 104.14 0) (unit 1)
     (in_bom yes) (on_board yes) (fields_autoplaced)
-    (property "Reference" "#PWR0183" (id 0) (at 115.57 110.49 0)
+    (property "Reference" "#PWR?" (id 0) (at 115.57 110.49 0)
       (effects (font (size 1.27 1.27)) hide)
     )
@@
   (symbol (lib_id "power:GND") (at 149.86 114.3 0) (unit 1)
     (in_bom yes) (on_board yes) (fields_autoplaced)
-    (property "Reference" "#PWR0186" (id 0) (at 149.86 120.65 0)
+    (property "Reference" "#PWR?" (id 0) (at 149.86 120.65 0)
       (effects (font (size 1.27 1.27)) hide)
     )
@@
   (symbol (lib_id "Device:R") (at 149.86 107.95 0) (unit 1)
     (in_bom yes) (on_board yes) (fields_autoplaced)
-    (property "Reference" "R77" (id 0) (at 152.4 106.6799 0)
-      (effects (font (size 1.27 1.27)) (justify left))
-    )
+    (property "Reference" "R?" (id 0) (at 152.4 106.6799 0)
+      (effects (font (size 1.27 1.27)) (justify left))
+    )
