File: JetsonCarrierBoard/dp-DESKTOP-4N3HF78.kicad_sch (KiCad schematic)
At the start: 23 parts, among them Q6 MMBT3904, Q7 MMBT3904, U17 TPD4E02B04DQA, U18 TPD4E02B04DQA, U19 TPD4E02B04DQA

Commit message: A ton
Parts:
- renumbered C76 to C?, C66 to C?, C75 to C?, C71 to C?, C73 to C?, C70 to C?, C68 to C?, C67 to C?, C69 to C?, C72 to C?, C74 to C?, Q6 to Q?, Q7 to Q?, R50 to R?, R54 to R?, R51 to R?, R48 to R?, R52 to R?, R49 to R?, R53 to R?, U18 to U?, U19 to U?, U17 to U?
Changed lines of the file:
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@@
   (symbol (lib_id "power:GND") (at 159.385 64.77 0) (unit 1)
     (in_bom yes) (on_board yes) (fields_autoplaced)
-    (property "Reference" "#PWR0144" (id 0) (at 159.385 71.12 0)
+    (property "Reference" "#PWR?" (id 0) (at 159.385 71.12 0)
       (effects (font (size 1.27 1.27)) hide)
     )
@@
   (symbol (lib_id "Device:C") (at 165.735 59.69 0) (unit 1)
     (in_bom yes) (on_board yes) (fields_autoplaced)
-    (property "Reference" "C76" (id 0) (at 168.656 58.8553 0)
+    (property "Reference" "C?" (id 0) (at 168.656 58.8553 0)
       (effects (font (size 1.27 1.27)) (justify left))
     )
@@
   (symbol (lib_id "power:GND") (at 142.875 62.23 0) (unit 1)
     (in_bom yes) (on_board yes) (fields_autoplaced)
-    (property "Reference" "#PWR0143" (id 0) (at 142.875 68.58 0)
+    (property "Reference" "#PWR?" (id 0) (at 142.875 68.58 0)
       (effects (font (size 1.27 1.27)) hide)
     )
@@
   (symbol (lib_id "Device:C") (at 140.97 85.725 90) (unit 1)
     (in_bom yes) (on_board yes)
-    (property "Reference" "C66" (id 0) (at 143.51 84.455 90))
+    (property "Reference" "C?" (id 0) (at 143.51 84.455 90))
     (property "Value" "0.1u" (id 1) (at 137.16 84.455 90))
     (property "Footprint" "" (id 2) (at 144.78 84.7598 0)
@@
   (symbol (lib_id "Device:R") (at 140.335 40.64 0) (unit 1)
     (in_bom yes) (on_board yes) (fields_autoplaced)
-    (property "Reference" "R50" (id 0) (at 142.113 39.8053 0)
+    (property "Reference" "R?" (id 0) (at 142.113 39.8053 0)
       (effects (font (size 1.27 1.27)) (justify left))
     )
@@
   (symbol (lib_id "Transistor_BJT:MMBT3904") (at 121.92 50.8 0) (mirror y) (unit 1)
     (in_bom yes) (on_board yes)
-    (property "Reference" "Q6" (id 0) (at 113.665 50.165 0)
+    (property "Reference" "Q?" (id 0) (at 113.665 50.165 0)
       (effects (font (size 1.27 1.27)) (justify left))
     )
@@
   (symbol (lib_id "Device:C") (at 152.4 132.08 90) (unit 1)
     (in_bom yes) (on_board yes)
-    (property "Reference" "C75" (id 0) (at 154.94 130.81 90))
+    (property "Reference" "C?" (id 0) (at 154.94 130.81 90))
     (property "Value" "0.1u" (id 1) (at 148.59 130.81 90))
     (property "Footprint" "" (id 2) (at 156.21 131.1148 0)
@@
   (symbol (lib_id "power:+1V8") (at 134.62 35.56 0) (unit 1)
     (in_bom yes) (on_board yes) (fields_autoplaced)
-    (property "Reference" "#PWR0142" (id 0) (at 134.62 39.37 0)
+    (property "Reference" "#PWR?" (id 0) (at 134.62 39.37 0)
       (effects (font (size 1.27 1.27)) hide)
     )
@@
   (symbol (lib_id "Device:C") (at 152.4 88.265 90) (unit 1)
     (in_bom yes) (on_board yes)
-    (property "Reference" "C71" (id 0) (at 154.94 86.995 90))
+    (property "Reference" "C?" (id 0) (at 154.94 86.995 90))
     (property "Value" "0.1u" (id 1) (at 148.59 86.995 90))
     (property "Footprint" "" (id 2) (at 156.21 87.2998 0)
@@
   (symbol (lib_id "Device:R") (at 161.29 92.075 0) (unit 1)
     (in_bom yes) (on_board yes) (fields_autoplaced)
-    (property "Reference" "R54" (id 0) (at 163.068 91.2403 0)
+    (property "Reference" "R?" (id 0) (at 163.068 91.2403 0)
       (effects (font (size 1.27 1.27)) (justify left))
     )
@@
   (symbol (lib_id "Device:C") (at 152.4 121.92 90) (unit 1)
     (in_bom yes) (on_board yes)
-    (property "Reference" "C73" (id 0) (at 154.94 120.65 90))
+    (property "Reference" "C?" (id 0) (at 154.94 120.65 90))
     (property "Value" "0.1u" (id 1) (at 148.59 120.65 90))
     (property "Footprint" "" (id 2) (at 156.21 120.9548 0)
@@
   (symbol (lib_id "power:GND") (at 161.29 97.155 0) (unit 1)
     (in_bom yes) (on_board yes) (fields_autoplaced)
-    (property "Reference" "#PWR0146" (id 0) (at 161.29 103.505 0)
+    (property "Reference" "#PWR?" (id 0) (at 161.29 103.505 0)
       (effects (font (size 1.27 1.27)) hide)
     )
@@
   (symbol (lib_id "Device:R") (at 153.035 59.69 0) (unit 1)
     (in_bom yes) (on_board yes) (fields_autoplaced)
-    (property "Reference" "R51" (id 0) (at 154.813 58.8553 0)
+    (property "Reference" "R?" (id 0) (at 154.813 58.8553 0)
       (effects (font (size 1.27 1.27)) (justify left))
     )
@@
   (symbol (lib_id "Device:R") (at 128.905 40.64 0) (unit 1)
     (in_bom yes) (on_board yes) (fields_autoplaced)
-    (property "Reference" "R48" (id 0) (at 130.683 39.8053 0)
+    (property "Reference" "R?" (id 0) (at 130.683 39.8053 0)
       (effects (font (size 1.27 1.27)) (justify left))
     )
@@
   (symbol (lib_id "Device:C") (at 140.97 129.54 90) (unit 1)
     (in_bom yes) (on_board yes)
-    (property "Reference" "C70" (id 0) (at 143.51 128.27 90))
+    (property "Reference" "C?" (id 0) (at 143.51 128.27 90))
     (property "Value" "0.1u" (id 1) (at 137.16 128.27 90))
     (property "Footprint" "" (id 2) (at 144.78 128.5748 0)
@@
   (symbol (lib_id "Device:R") (at 159.385 55.88 90) (unit 1)
     (in_bom yes) (on_board yes) (fields_autoplaced)
-    (property "Reference" "R52" (id 0) (at 159.385 51.1642 90))
+    (property "Reference" "R?" (id 0) (at 159.385 51.1642 90))
     (property "Value" "100k" (id 1) (at 159.385 53.7011 90))
     (property "Footprint" "" (id 2) (at 159.385 57.658 90)
@@
   (symbol (lib_id "power:GND") (at 119.38 57.15 0) (unit 1)
     (in_bom yes) (on_board yes) (fields_autoplaced)
-    (property "Reference" "#PWR0141" (id 0) (at 119.38 63.5 0)
+    (property "Reference" "#PWR?" (id 0) (at 119.38 63.5 0)
       (effects (font (size 1.27 1.27)) hide)
     )
@@
   (symbol (lib_id "Device:C") (at 140.97 119.38 90) (unit 1)
     (in_bom yes) (on_board yes)
-    (property "Reference" "C68" (id 0) (at 143.51 118.11 90))
+    (property "Reference" "C?" (id 0) (at 143.51 118.11 90))
     (property "Value" "0.1u" (id 1) (at 137.16 118.11 90))
     (property "Footprint" "" (id 2) (at 144.78 118.4148 0)
@@
   (symbol (lib_id "Device:R") (at 134.62 50.8 90) (unit 1)
     (in_bom yes) (on_board yes) (fields_autoplaced)
-    (property "Reference" "R49" (id 0) (at 134.62 46.0842 90))
+    (property "Reference" "R?" (id 0) (at 134.62 46.0842 90))
     (property "Value" "5.1k" (id 1) (at 134.62 48.6211 90))
     (property "Footprint" "" (id 2) (at 134.62 52.578 90)
@@
   (symbol (lib_id "power:GND") (at 177.8 105.41 0) (unit 1)
     (in_bom yes) (on_board yes) (fields_autoplaced)
-    (property "Reference" "#PWR0148" (id 0) (at 177.8 111.76 0)
+    (property "Reference" "#PWR?" (id 0) (at 177.8 111.76 0)
       (effects (font (size 1.27 1.27)) hide)
     )
@@
   (symbol (lib_id "power:+3.3V") (at 161.29 76.835 0) (unit 1)
     (in_bom yes) (on_board yes) (fields_autoplaced)
-    (property "Reference" "#PWR0145" (id 0) (at 161.29 80.645 0)
+    (property "Reference" "#PWR?" (id 0) (at 161.29 80.645 0)
       (effects (font (size 1.27 1.27)) hide)
     )
@@
   (symbol (lib_id "Power_Protection:TPD4E02B04DQA") (at 175.895 143.51 0) (unit 1)
     (in_bom yes) (on_board yes)
-    (property "Reference" "U18" (id 0) (at 184.15 145.415 0)
+    (property "Reference" "U?" (id 0) (at 184.15 145.415 0)
       (effects (font (size 1.27 1.27)) (justify left))
     )
@@
   (symbol (lib_id "Device:C") (at 140.97 114.3 90) (unit 1)
     (in_bom yes) (on_board yes)
-    (property "Reference" "C67" (id 0) (at 143.51 113.03 90))
+    (property "Reference" "C?" (id 0) (at 143.51 113.03 90))
     (property "Value" "0.1u" (id 1) (at 137.16 113.03 90))
     (property "Footprint" "" (id 2) (at 144.78 113.3348 0)
@@
   (symbol (lib_id "Device:C") (at 140.97 124.46 90) (unit 1)
     (in_bom yes) (on_board yes)
-    (property "Reference" "C69" (id 0) (at 143.51 123.19 90))
+    (property "Reference" "C?" (id 0) (at 143.51 123.19 90))
     (property "Value" "0.1u" (id 1) (at 137.16 123.19 90))
     (property "Footprint" "" (id 2) (at 144.78 123.4948 0)
@@
   (symbol (lib_id "Power_Protection:TPD4E02B04DQA") (at 177.8 99.06 0) (unit 1)
     (in_bom yes) (on_board yes)
-    (property "Reference" "U19" (id 0) (at 186.055 100.965 0)
+    (property "Reference" "U?" (id 0) (at 186.055 100.965 0)
       (effects (font (size 1.27 1.27)) (justify left))
     )
@@
   (symbol (lib_id "Power_Protection:TPD4E02B04DQA") (at 161.925 143.51 0) (unit 1)
     (in_bom yes) (on_board yes)
-    (property "Reference" "U17" (id 0) (at 150.495 145.415 0)
+    (property "Reference" "U?" (id 0) (at 150.495 145.415 0)
       (effects (font (size 1.27 1.27)) (justify left))
     )
@@
   (symbol (lib_id "Transistor_BJT:MMBT3904") (at 145.415 55.88 0) (mirror y) (unit 1)
     (in_bom yes) (on_board yes)
-    (property "Reference" "Q7" (id 0) (at 137.16 55.245 0)
+    (property "Reference" "Q?" (id 0) (at 137.16 55.245 0)
       (effects (font (size 1.27 1.27)) (justify left))
     )
@@
   (symbol (lib_id "power:GND") (at 168.91 149.86 0) (unit 1)
     (in_bom yes) (on_board yes) (fields_autoplaced)
-    (property "Reference" "#PWR0147" (id 0) (at 168.91 156.21 0)
+    (property "Reference" "#PWR?" (id 0) (at 168.91 156.21 0)
       (effects (font (size 1.27 1.27)) hide)
     )
@@
   (symbol (lib_id "Device:R") (at 161.29 81.915 0) (unit 1)
     (in_bom yes) (on_board yes) (fields_autoplaced)
-    (property "Reference" "R53" (id 0) (at 163.068 81.0803 0)
+    (property "Reference" "R?" (id 0) (at 163.068 81.0803 0)
       (effects (font (size 1.27 1.27)) (justify left))
     )
@@
   (symbol (lib_id "Device:C") (at 152.4 116.84 90) (unit 1)
     (in_bom yes) (on_board yes)
-    (property "Reference" "C72" (id 0) (at 154.94 115.57 90))
+    (property "Reference" "C?" (id 0) (at 154.94 115.57 90))
     (property "Value" "0.1u" (id 1) (at 148.59 115.57 90))
     (property "Footprint" "" (id 2) (at 156.21 115.8748 0)
@@
   (symbol (lib_id "Device:C") (at 152.4 127 90) (unit 1)
     (in_bom yes) (on_board yes)
-    (property "Reference" "C74" (id 0) (at 154.94 125.73 90))
+    (property "Reference" "C?" (id 0) (at 154.94 125.73 90))
     (property "Value" "0.1u" (id 1) (at 148.59 125.73 90))
     (property "Footprint" "" (id 2) (at 156.21 126.0348 0)
