File: JetsonCarrierBoard/fan_debug-DESKTOP-4N3HF78.kicad_sch (KiCad schematic)
At the start: 17 parts, among them J10 Conn_01x04, J9 Conn_01x08, Q12 DMN24H3D5L, Q13 DMN24H3D5L, U26 SN74LVC1T45DBV

Commit message: A ton
Parts:
- D?: renamed from D32; value D_TPD -> D_TVS
- D?: renamed from D33; value D_TPD -> D_TVS
- D?: renamed from D34; value D_TPD -> D_TVS
- renumbered C88 to C?, C89 to C?, D35 to D?, J9 to J?, J10 to J?, Q13 to Q?, Q12 to Q?, R82 to R?, R81 to R?, R85 to R?, R80 to R?, R83 to R?, R84 to R?, U26 to U?
