File: JetsonCarrierBoard/gpio-DESKTOP-4N3HF78.kicad_sch (KiCad schematic)
At the start: 19 parts, among them J5 Conn_02x13_Odd_Even, J6 Conn_01x04, Q5 NTS4101PT1G, U14 TXB0108DQSR, U15 TXB0108DQSR, U16 NST45010MW6T1G

Commit message: A ton
Parts:
- D?: renamed from D24; value D_LES -> D_TVS
- D?: renamed from D25; value D_LES -> D_TVS
- renumbered C64 to C?, C62 to C?, C63 to C?, C65 to C?, J5 to J?, J6 to J?, Q5 to Q?, R43 to R?, R44 to R?, R41 to R?, R47 to R?, R42 to R?, R46 to R?, R45 to R?, U15 to U?, U16 to U?, U14 to U?
