File: JetsonCarrierBoard/imu-DESKTOP-4N3HF78.kicad_sch (KiCad schematic)
At the start: 5 parts, among them U13 ICM-20602

Commit message: A ton
Parts:
- renumbered C61 to C?, C60 to C?, C58 to C?, C59 to C?, U13 to U?
Changed lines of the file:
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@@
   (symbol (lib_id "power:GND") (at 166.37 90.17 0) (unit 1)
     (in_bom yes) (on_board yes) (fields_autoplaced)
-    (property "Reference" "#PWR0105" (id 0) (at 166.37 96.52 0)
+    (property "Reference" "#PWR?" (id 0) (at 166.37 96.52 0)
       (effects (font (size 1.27 1.27)) hide)
     )
@@
   (symbol (lib_id "power:GND") (at 167.64 102.87 90) (unit 1)
     (in_bom yes) (on_board yes) (fields_autoplaced)
-    (property "Reference" "#PWR0106" (id 0) (at 173.99 102.87 0)
+    (property "Reference" "#PWR?" (id 0) (at 173.99 102.87 0)
       (effects (font (size 1.27 1.27)) hide)
     )
@@
   (symbol (lib_id "Device:C") (at 167.64 109.22 0) (unit 1)
     (in_bom yes) (on_board yes) (fields_autoplaced)
-    (property "Reference" "C61" (id 0) (at 171.45 107.9499 0)
+    (property "Reference" "C?" (id 0) (at 171.45 107.9499 0)
       (effects (font (size 1.27 1.27)) (justify left))
     )
@@
   (symbol (lib_id "power:+1V8") (at 132.08 80.01 0) (unit 1)
     (in_bom yes) (on_board yes) (fields_autoplaced)
-    (property "Reference" "#PWR0102" (id 0) (at 132.08 83.82 0)
+    (property "Reference" "#PWR?" (id 0) (at 132.08 83.82 0)
       (effects (font (size 1.27 1.27)) hide)
     )
@@
   (symbol (lib_id "Device:C") (at 160.02 87.63 90) (unit 1)
     (in_bom yes) (on_board yes)
-    (property "Reference" "C60" (id 0) (at 160.02 81.28 90))
+    (property "Reference" "C?" (id 0) (at 160.02 81.28 90))
     (property "Value" "10n" (id 1) (at 160.02 83.82 90))
     (property "Footprint" "" (id 2) (at 163.83 86.6648 0)
@@
   (symbol (lib_id "power:GND") (at 132.08 90.17 0) (unit 1)
     (in_bom yes) (on_board yes) (fields_autoplaced)
-    (property "Reference" "#PWR0103" (id 0) (at 132.08 96.52 0)
+    (property "Reference" "#PWR?" (id 0) (at 132.08 96.52 0)
       (effects (font (size 1.27 1.27)) hide)
     )
@@
   (symbol (lib_id "power:GND") (at 149.86 118.11 0) (unit 1)
     (in_bom yes) (on_board yes) (fields_autoplaced)
-    (property "Reference" "#PWR0104" (id 0) (at 149.86 124.46 0)
+    (property "Reference" "#PWR?" (id 0) (at 149.86 124.46 0)
       (effects (font (size 1.27 1.27)) hide)
     )
@@
   (symbol (lib_id "Device:C") (at 125.73 86.36 0) (unit 1)
     (in_bom yes) (on_board yes) (fields_autoplaced)
-    (property "Reference" "C58" (id 0) (at 129.54 85.0899 0)
+    (property "Reference" "C?" (id 0) (at 129.54 85.0899 0)
       (effects (font (size 1.27 1.27)) (justify left))
     )
@@
   (symbol (lib_id "power:GND") (at 167.64 115.57 0) (unit 1)
     (in_bom yes) (on_board yes) (fields_autoplaced)
-    (property "Reference" "#PWR0107" (id 0) (at 167.64 121.92 0)
+    (property "Reference" "#PWR?" (id 0) (at 167.64 121.92 0)
       (effects (font (size 1.27 1.27)) hide)
     )
@@
   (symbol (lib_id "Sensor_Motion:ICM-20602") (at 149.86 102.87 0) (unit 1)
     (in_bom yes) (on_board yes) (fields_autoplaced)
-    (property "Reference" "U13" (id 0) (at 151.8794 115.57 0)
+    (property "Reference" "U?" (id 0) (at 151.8794 115.57 0)
       (effects (font (size 1.27 1.27)) (justify left))
     )
@@
   (symbol (lib_id "Device:C") (at 138.43 86.36 0) (unit 1)
     (in_bom yes) (on_board yes) (fields_autoplaced)
-    (property "Reference" "C59" (id 0) (at 142.24 85.0899 0)
+    (property "Reference" "C?" (id 0) (at 142.24 85.0899 0)
       (effects (font (size 1.27 1.27)) (justify left))
     )
