File: JetsonCarrierBoard/ldoAo-DESKTOP-4N3HF78.kicad_sch (KiCad schematic)
At the start: 4 parts, among them U24 TLV707, U25 MIC5528

Commit message: A ton
Parts:
- renumbered C80 to C?, C81 to C?, U25 to U?, U24 to U?
Changed lines of the file:
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@@
   (symbol (lib_id "Device:C") (at 154.94 100.203 0) (unit 1)
     (in_bom yes) (on_board yes) (fields_autoplaced)
-    (property "Reference" "C80" (id 0) (at 157.861 99.3683 0)
+    (property "Reference" "C?" (id 0) (at 157.861 99.3683 0)
       (effects (font (size 1.27 1.27)) (justify left))
     )
@@
   (symbol (lib_id "power:+5V") (at 169.545 95.123 0) (unit 1)
     (in_bom yes) (on_board yes) (fields_autoplaced)
-    (property "Reference" "#PWR0180" (id 0) (at 169.545 98.933 0)
+    (property "Reference" "#PWR?" (id 0) (at 169.545 98.933 0)
       (effects (font (size 1.27 1.27)) hide)
     )
@@
   (symbol (lib_id "Voltage_Regulators_Linear:MIC5528") (at 179.705 93.853 0) (unit 1)
     (in_bom yes) (on_board yes) (fields_autoplaced)
-    (property "Reference" "U25" (id 0) (at 180.34 90.204 0))
+    (property "Reference" "U?" (id 0) (at 180.34 90.204 0))
     (property "Value" "MIC5528" (id 1) (at 180.34 92.7409 0))
     (property "Footprint" "" (id 2) (at 179.705 93.853 0)
@@
   (symbol (lib_id "power:+1V8") (at 124.46 92.583 0) (unit 1)
     (in_bom yes) (on_board yes) (fields_autoplaced)
-    (property "Reference" "#PWR0178" (id 0) (at 124.46 96.393 0)
+    (property "Reference" "#PWR?" (id 0) (at 124.46 96.393 0)
       (effects (font (size 1.27 1.27)) hide)
     )
@@
   (symbol (lib_id "power:GND") (at 193.04 104.648 0) (unit 1)
     (in_bom yes) (on_board yes) (fields_autoplaced)
-    (property "Reference" "#PWR0182" (id 0) (at 193.04 110.998 0)
+    (property "Reference" "#PWR?" (id 0) (at 193.04 110.998 0)
       (effects (font (size 1.27 1.27)) hide)
     )
@@
   (symbol (lib_id "Voltage_Regulators_Linear:TLV707") (at 111.76 88.773 0) (unit 1)
     (in_bom yes) (on_board yes) (fields_autoplaced)
-    (property "Reference" "U24" (id 0) (at 111.76 86.394 0))
+    (property "Reference" "U?" (id 0) (at 111.76 86.394 0))
     (property "Value" "TLV707" (id 1) (at 111.76 88.9309 0))
     (property "Footprint" "" (id 2) (at 111.76 88.773 0)
@@
   (symbol (lib_id "Device:C") (at 193.04 98.933 0) (unit 1)
     (in_bom yes) (on_board yes) (fields_autoplaced)
-    (property "Reference" "C81" (id 0) (at 195.961 98.0983 0)
+    (property "Reference" "C?" (id 0) (at 195.961 98.0983 0)
       (effects (font (size 1.27 1.27)) (justify left))
     )
@@
   (symbol (lib_id "power:+3.3VA") (at 193.04 93.218 0) (unit 1)
     (in_bom yes) (on_board yes) (fields_autoplaced)
-    (property "Reference" "#PWR0181" (id 0) (at 193.04 97.028 0)
+    (property "Reference" "#PWR?" (id 0) (at 193.04 97.028 0)
       (effects (font (size 1.27 1.27)) hide)
     )
@@
   (symbol (lib_id "power:+3.3V") (at 99.06 92.583 0) (unit 1)
     (in_bom yes) (on_board yes) (fields_autoplaced)
-    (property "Reference" "#PWR0176" (id 0) (at 99.06 96.393 0)
+    (property "Reference" "#PWR?" (id 0) (at 99.06 96.393 0)
       (effects (font (size 1.27 1.27)) hide)
     )
@@
   (symbol (lib_id "power:GND") (at 111.76 109.093 0) (unit 1)
     (in_bom yes) (on_board yes) (fields_autoplaced)
-    (property "Reference" "#PWR0177" (id 0) (at 111.76 115.443 0)
+    (property "Reference" "#PWR?" (id 0) (at 111.76 115.443 0)
       (effects (font (size 1.27 1.27)) hide)
     )
@@
   (symbol (lib_id "power:GND") (at 154.94 105.283 0) (unit 1)
     (in_bom yes) (on_board yes) (fields_autoplaced)
-    (property "Reference" "#PWR0179" (id 0) (at 154.94 111.633 0)
+    (property "Reference" "#PWR?" (id 0) (at 154.94 111.633 0)
       (effects (font (size 1.27 1.27)) hide)
     )
