File: JetsonCarrierBoard/m2ssd-DESKTOP-4N3HF78.kicad_sch (KiCad schematic)
At the start: 14 parts, among them J2 Bus_M.2_Socket_M, U4 OSC32.768

Commit message: A ton
Parts:
- renumbered C27 to C?, C24 to C?, C34 to C?, C32 to C?, C30 to C?, C29 to C?, C26 to C?, C25 to C?, C28 to C?, C31 to C?, C33 to C?, H3 to H?, J2 to J?, U4 to U?
Changed lines of the file:
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@@
   (symbol (lib_id "Mechanical:MountingHole_Pad") (at 91.44 128.27 0) (unit 1)
     (in_bom yes) (on_board yes) (fields_autoplaced)
-    (property "Reference" "H3" (id 0) (at 93.98 125.7299 0)
+    (property "Reference" "H?" (id 0) (at 93.98 125.7299 0)
       (effects (font (size 1.27 1.27)) (justify left))
     )
@@
   (symbol (lib_id "Crystals:OSC32.768") (at 74.93 69.85 0) (unit 1)
     (in_bom yes) (on_board yes) (fields_autoplaced)
-    (property "Reference" "U4" (id 0) (at 74.93 64.77 0))
+    (property "Reference" "U?" (id 0) (at 74.93 64.77 0))
     (property "Value" "OSC32.768" (id 1) (at 74.93 67.31 0))
     (property "Footprint" "" (id 2) (at 74.93 69.85 0)
@@
   (symbol (lib_id "power:GND") (at 181.61 149.86 0) (unit 1)
     (in_bom yes) (on_board yes) (fields_autoplaced)
-    (property "Reference" "#PWR036" (id 0) (at 181.61 156.21 0)
+    (property "Reference" "#PWR?" (id 0) (at 181.61 156.21 0)
       (effects (font (size 1.27 1.27)) hide)
     )
@@
   (symbol (lib_id "Device:C") (at 139.7 86.36 90) (unit 1)
     (in_bom yes) (on_board yes)
-    (property "Reference" "C27" (id 0) (at 142.24 85.09 90))
+    (property "Reference" "C?" (id 0) (at 142.24 85.09 90))
     (property "Value" "0.22u" (id 1) (at 135.89 85.09 90))
     (property "Footprint" "" (id 2) (at 143.51 85.3948 0)
@@
   (symbol (lib_id "power:GND") (at 91.44 133.35 0) (unit 1)
     (in_bom yes) (on_board yes) (fields_autoplaced)
-    (property "Reference" "#PWR034" (id 0) (at 91.44 139.7 0)
+    (property "Reference" "#PWR?" (id 0) (at 91.44 139.7 0)
       (effects (font (size 1.27 1.27)) hide)
     )
@@
   (symbol (lib_id "Device:C") (at 86.36 57.15 0) (unit 1)
     (in_bom yes) (on_board yes) (fields_autoplaced)
-    (property "Reference" "C24" (id 0) (at 90.17 55.8799 0)
+    (property "Reference" "C?" (id 0) (at 90.17 55.8799 0)
       (effects (font (size 1.27 1.27)) (justify left))
     )
@@
   (symbol (lib_id "power:+3.3V") (at 78.74 53.34 0) (unit 1)
     (in_bom yes) (on_board yes) (fields_autoplaced)
-    (property "Reference" "#PWR032" (id 0) (at 78.74 57.15 0)
+    (property "Reference" "#PWR?" (id 0) (at 78.74 57.15 0)
       (effects (font (size 1.27 1.27)) hide)
     )
@@
   (symbol (lib_id "power:GND") (at 64.77 80.01 0) (unit 1)
     (in_bom yes) (on_board yes) (fields_autoplaced)
-    (property "Reference" "#PWR031" (id 0) (at 64.77 86.36 0)
+    (property "Reference" "#PWR?" (id 0) (at 64.77 86.36 0)
       (effects (font (size 1.27 1.27)) hide)
     )
@@
   (symbol (lib_id "Device:C") (at 222.25 60.96 0) (unit 1)
     (in_bom yes) (on_board yes) (fields_autoplaced)
-    (property "Reference" "C34" (id 0) (at 226.06 59.6899 0)
+    (property "Reference" "C?" (id 0) (at 226.06 59.6899 0)
       (effects (font (size 1.27 1.27)) (justify left))
     )
@@
   (symbol (lib_id "Device:C") (at 148.59 99.06 90) (unit 1)
     (in_bom yes) (on_board yes)
-    (property "Reference" "C32" (id 0) (at 151.13 97.79 90))
+    (property "Reference" "C?" (id 0) (at 151.13 97.79 90))
     (property "Value" "0.22u" (id 1) (at 144.78 97.79 90))
     (property "Footprint" "" (id 2) (at 152.4 98.0948 0)
@@
   (symbol (lib_id "power:GND") (at 215.9 67.31 0) (unit 1)
     (in_bom yes) (on_board yes) (fields_autoplaced)
-    (property "Reference" "#PWR038" (id 0) (at 215.9 73.66 0)
+    (property "Reference" "#PWR?" (id 0) (at 215.9 73.66 0)
       (effects (font (size 1.27 1.27)) hide)
     )
@@
   (symbol (lib_id "power:+3.3V") (at 215.9 54.61 0) (unit 1)
     (in_bom yes) (on_board yes) (fields_autoplaced)
-    (property "Reference" "#PWR037" (id 0) (at 215.9 58.42 0)
+    (property "Reference" "#PWR?" (id 0) (at 215.9 58.42 0)
       (effects (font (size 1.27 1.27)) hide)
     )
@@
   (symbol (lib_id "Device:C") (at 148.59 78.74 90) (unit 1)
     (in_bom yes) (on_board yes)
-    (property "Reference" "C30" (id 0) (at 151.13 77.47 90))
+    (property "Reference" "C?" (id 0) (at 151.13 77.47 90))
     (property "Value" "0.22u" (id 1) (at 144.78 77.47 90))
     (property "Footprint" "" (id 2) (at 152.4 77.7748 0)
@@
   (symbol (lib_id "Device:C") (at 148.59 68.58 90) (unit 1)
     (in_bom yes) (on_board yes)
-    (property "Reference" "C29" (id 0) (at 151.13 67.31 90))
+    (property "Reference" "C?" (id 0) (at 151.13 67.31 90))
     (property "Value" "0.22u" (id 1) (at 144.78 67.31 90))
     (property "Footprint" "" (id 2) (at 152.4 67.6148 0)
@@
   (symbol (lib_id "power:+3.3V") (at 181.61 48.26 0) (unit 1)
     (in_bom yes) (on_board yes) (fields_autoplaced)
-    (property "Reference" "#PWR035" (id 0) (at 181.61 52.07 0)
+    (property "Reference" "#PWR?" (id 0) (at 181.61 52.07 0)
       (effects (font (size 1.27 1.27)) hide)
     )
@@
   (symbol (lib_id "Connector:Bus_M.2_Socket_M") (at 181.61 99.06 0) (unit 1)
     (in_bom yes) (on_board yes) (fields_autoplaced)
-    (property "Reference" "J2" (id 0) (at 183.6294 48.26 0)
+    (property "Reference" "J?" (id 0) (at 183.6294 48.26 0)
       (effects (font (size 1.27 1.27)) (justify left))
     )
@@
   (symbol (lib_id "Device:C") (at 139.7 76.2 90) (unit 1)
     (in_bom yes) (on_board yes)
-    (property "Reference" "C26" (id 0) (at 142.24 74.93 90))
+    (property "Reference" "C?" (id 0) (at 142.24 74.93 90))
     (property "Value" "0.22u" (id 1) (at 135.89 74.93 90))
     (property "Footprint" "" (id 2) (at 143.51 75.2348 0)
@@
   (symbol (lib_id "Device:C") (at 139.7 66.04 90) (unit 1)
     (in_bom yes) (on_board yes)
-    (property "Reference" "C25" (id 0) (at 142.24 64.77 90))
+    (property "Reference" "C?" (id 0) (at 142.24 64.77 90))
     (property "Value" "0.22u" (id 1) (at 135.89 64.77 90))
     (property "Footprint" "" (id 2) (at 143.51 65.0748 0)
@@
   (symbol (lib_id "power:GND") (at 86.36 63.5 0) (unit 1)
     (in_bom yes) (on_board yes) (fields_autoplaced)
-    (property "Reference" "#PWR033" (id 0) (at 86.36 69.85 0)
+    (property "Reference" "#PWR?" (id 0) (at 86.36 69.85 0)
       (effects (font (size 1.27 1.27)) hide)
     )
@@
   (symbol (lib_id "Device:C") (at 139.7 96.52 90) (unit 1)
     (in_bom yes) (on_board yes)
-    (property "Reference" "C28" (id 0) (at 142.24 95.25 90))
+    (property "Reference" "C?" (id 0) (at 142.24 95.25 90))
     (property "Value" "0.22u" (id 1) (at 135.89 95.25 90))
     (property "Footprint" "" (id 2) (at 143.51 95.5548 0)
@@
   (symbol (lib_id "Device:C") (at 148.59 88.9 90) (unit 1)
     (in_bom yes) (on_board yes)
-    (property "Reference" "C31" (id 0) (at 151.13 87.63 90))
+    (property "Reference" "C?" (id 0) (at 151.13 87.63 90))
     (property "Value" "0.22u" (id 1) (at 144.78 87.63 90))
     (property "Footprint" "" (id 2) (at 152.4 87.9348 0)
@@
   (symbol (lib_id "Device:C") (at 209.55 60.96 0) (unit 1)
     (in_bom yes) (on_board yes) (fields_autoplaced)
-    (property "Reference" "C33" (id 0) (at 213.36 59.6899 0)
-      (effects (font (size 1.27 1.27)) (justify left))
-    )
+    (property "Reference" "C?" (id 0) (at 213.36 59.6899 0)
+      (effects (font (size 1.27 1.27)) (justify left))
+    )
