File: JetsonCarrierBoard/m2wifi-DESKTOP-4N3HF78.kicad_sch (KiCad schematic)
At the start: 15 parts, among them J3 Bus_M.2_Socket_E, Q3 DMN24H3D5L, Q4 DMN24H3D5L

Commit message: A ton
Parts:
- renumbered C35 to C?, C40 to C?, C39 to C?, C36 to C?, C38 to C?, C37 to C?, H4 to H?, J3 to J?, Q3 to Q?, Q4 to Q?, R28 to R?, R26 to R?, R27 to R?, R24 to R?, R25 to R?
Changed lines of the file:
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@@
   (symbol (lib_id "power:+3.3V") (at 248.92 105.41 0) (unit 1)
     (in_bom yes) (on_board yes) (fields_autoplaced)
-    (property "Reference" "#PWR047" (id 0) (at 248.92 109.22 0)
+    (property "Reference" "#PWR?" (id 0) (at 248.92 109.22 0)
       (effects (font (size 1.27 1.27)) hide)
     )
@@
   (symbol (lib_id "power:GND") (at 248.92 50.8 0) (unit 1)
     (in_bom yes) (on_board yes) (fields_autoplaced)
-    (property "Reference" "#PWR044" (id 0) (at 248.92 57.15 0)
+    (property "Reference" "#PWR?" (id 0) (at 248.92 57.15 0)
       (effects (font (size 1.27 1.27)) hide)
     )
@@
   (symbol (lib_id "Device:C") (at 102.87 67.31 90) (unit 1)
     (in_bom yes) (on_board yes)
-    (property "Reference" "C35" (id 0) (at 105.41 66.04 90))
+    (property "Reference" "C?" (id 0) (at 105.41 66.04 90))
     (property "Value" "0.1u" (id 1) (at 99.06 66.04 90))
     (property "Footprint" "" (id 2) (at 106.68 66.3448 0)
@@
   (symbol (lib_id "Device:C") (at 156.21 46.99 90) (unit 1)
     (in_bom yes) (on_board yes) (fields_autoplaced)
-    (property "Reference" "C40" (id 0) (at 156.21 41.1312 90))
+    (property "Reference" "C?" (id 0) (at 156.21 41.1312 90))
     (property "Value" "10u" (id 1) (at 156.21 43.6681 90))
     (property "Footprint" "" (id 2) (at 160.02 46.0248 0)
@@
   (symbol (lib_id "Device:C") (at 156.21 36.83 90) (unit 1)
     (in_bom yes) (on_board yes) (fields_autoplaced)
-    (property "Reference" "C39" (id 0) (at 156.21 30.9712 90))
+    (property "Reference" "C?" (id 0) (at 156.21 30.9712 90))
     (property "Value" "0.1u" (id 1) (at 156.21 33.5081 90))
     (property "Footprint" "" (id 2) (at 160.02 35.8648 0)
@@
   (symbol (lib_id "Device:C") (at 113.03 64.77 90) (unit 1)
     (in_bom yes) (on_board yes)
-    (property "Reference" "C36" (id 0) (at 115.57 63.5 90))
+    (property "Reference" "C?" (id 0) (at 115.57 63.5 90))
     (property "Value" "0.1u" (id 1) (at 109.22 63.5 90))
     (property "Footprint" "" (id 2) (at 116.84 63.8048 0)
@@
   (symbol (lib_id "power:GND") (at 134.62 41.91 270) (unit 1)
     (in_bom yes) (on_board yes) (fields_autoplaced)
-    (property "Reference" "#PWR040" (id 0) (at 128.27 41.91 0)
+    (property "Reference" "#PWR?" (id 0) (at 128.27 41.91 0)
       (effects (font (size 1.27 1.27)) hide)
     )
@@
   (symbol (lib_id "Device:R") (at 248.92 111.76 0) (unit 1)
     (in_bom yes) (on_board yes)
-    (property "Reference" "R28" (id 0) (at 250.698 110.9253 0)
+    (property "Reference" "R?" (id 0) (at 250.698 110.9253 0)
       (effects (font (size 1.27 1.27)) (justify left))
     )
@@
   (symbol (lib_id "Transistor_FET:DMN24H3D5L") (at 246.38 83.82 0) (unit 1)
     (in_bom yes) (on_board yes) (fields_autoplaced)
-    (property "Reference" "Q3" (id 0) (at 252.73 82.5499 0)
+    (property "Reference" "Q?" (id 0) (at 252.73 82.5499 0)
       (effects (font (size 1.27 1.27)) (justify left))
     )
@@
   (symbol (lib_id "Mechanical:MountingHole_Pad") (at 248.92 45.72 0) (unit 1)
     (in_bom yes) (on_board yes) (fields_autoplaced)
-    (property "Reference" "H4" (id 0) (at 251.46 43.1799 0)
+    (property "Reference" "H?" (id 0) (at 251.46 43.1799 0)
       (effects (font (size 1.27 1.27)) (justify left))
     )
@@
   (symbol (lib_id "power:GND") (at 248.92 91.44 0) (unit 1)
     (in_bom yes) (on_board yes) (fields_autoplaced)
-    (property "Reference" "#PWR046" (id 0) (at 248.92 97.79 0)
+    (property "Reference" "#PWR?" (id 0) (at 248.92 97.79 0)
       (effects (font (size 1.27 1.27)) hide)
     )
@@
   (symbol (lib_id "Device:R") (at 120.65 48.26 0) (unit 1)
     (in_bom yes) (on_board yes)
-    (property "Reference" "R26" (id 0) (at 122.428 47.4253 0)
+    (property "Reference" "R?" (id 0) (at 122.428 47.4253 0)
       (effects (font (size 1.27 1.27)) (justify left))
     )
@@
   (symbol (lib_id "power:+3.3V") (at 248.92 66.04 0) (unit 1)
     (in_bom yes) (on_board yes) (fields_autoplaced)
-    (property "Reference" "#PWR045" (id 0) (at 248.92 69.85 0)
+    (property "Reference" "#PWR?" (id 0) (at 248.92 69.85 0)
       (effects (font (size 1.27 1.27)) hide)
     )
@@
   (symbol (lib_id "power:GND") (at 162.56 41.91 90) (unit 1)
     (in_bom yes) (on_board yes) (fields_autoplaced)
-    (property "Reference" "#PWR043" (id 0) (at 168.91 41.91 0)
+    (property "Reference" "#PWR?" (id 0) (at 168.91 41.91 0)
       (effects (font (size 1.27 1.27)) hide)
     )
@@
   (symbol (lib_id "Device:R") (at 248.92 72.39 0) (unit 1)
     (in_bom yes) (on_board yes)
-    (property "Reference" "R27" (id 0) (at 250.698 71.5553 0)
+    (property "Reference" "R?" (id 0) (at 250.698 71.5553 0)
       (effects (font (size 1.27 1.27)) (justify left))
     )
@@
   (symbol (lib_id "Device:R") (at 107.95 48.26 0) (unit 1)
     (in_bom yes) (on_board yes)
-    (property "Reference" "R24" (id 0) (at 109.728 47.4253 0)
+    (property "Reference" "R?" (id 0) (at 109.728 47.4253 0)
       (effects (font (size 1.27 1.27)) (justify left))
     )
@@
   (symbol (lib_id "Device:C") (at 140.97 46.99 90) (unit 1)
     (in_bom yes) (on_board yes) (fields_autoplaced)
-    (property "Reference" "C38" (id 0) (at 140.97 41.1312 90))
+    (property "Reference" "C?" (id 0) (at 140.97 41.1312 90))
     (property "Value" "10u" (id 1) (at 140.97 43.6681 90))
     (property "Footprint" "" (id 2) (at 144.78 46.0248 0)
@@
   (symbol (lib_id "Transistor_FET:DMN24H3D5L") (at 246.38 123.19 0) (unit 1)
     (in_bom yes) (on_board yes) (fields_autoplaced)
-    (property "Reference" "Q4" (id 0) (at 252.73 121.9199 0)
+    (property "Reference" "Q?" (id 0) (at 252.73 121.9199 0)
       (effects (font (size 1.27 1.27)) (justify left))
     )
@@
   (symbol (lib_id "Device:R") (at 114.3 48.26 0) (unit 1)
     (in_bom yes) (on_board yes)
-    (property "Reference" "R25" (id 0) (at 116.078 47.4253 0)
+    (property "Reference" "R?" (id 0) (at 116.078 47.4253 0)
       (effects (font (size 1.27 1.27)) (justify left))
     )
@@
   (symbol (lib_id "Device:C") (at 140.97 36.83 90) (unit 1)
     (in_bom yes) (on_board yes) (fields_autoplaced)
-    (property "Reference" "C37" (id 0) (at 140.97 30.9712 90))
+    (property "Reference" "C?" (id 0) (at 140.97 30.9712 90))
     (property "Value" "0.1u" (id 1) (at 140.97 33.5081 90))
     (property "Footprint" "" (id 2) (at 144.78 35.8648 0)
@@
   (symbol (lib_id "power:GND") (at 248.92 130.81 0) (unit 1)
     (in_bom yes) (on_board yes) (fields_autoplaced)
-    (property "Reference" "#PWR048" (id 0) (at 248.92 137.16 0)
+    (property "Reference" "#PWR?" (id 0) (at 248.92 137.16 0)
       (effects (font (size 1.27 1.27)) hide)
     )
@@
   (symbol (lib_id "power:GND") (at 148.59 148.59 0) (unit 1)
     (in_bom yes) (on_board yes) (fields_autoplaced)
-    (property "Reference" "#PWR042" (id 0) (at 148.59 154.94 0)
+    (property "Reference" "#PWR?" (id 0) (at 148.59 154.94 0)
       (effects (font (size 1.27 1.27)) hide)
     )
@@
   (symbol (lib_id "Connector:Bus_M.2_Socket_E") (at 148.59 97.79 0) (unit 1)
     (in_bom yes) (on_board yes) (fields_autoplaced)
-    (property "Reference" "J3" (id 0) (at 150.6094 48.3702 0)
+    (property "Reference" "J?" (id 0) (at 150.6094 48.3702 0)
       (effects (font (size 1.27 1.27)) (justify left))
     )
@@
   (symbol (lib_id "power:+3.3V") (at 114.3 41.91 0) (unit 1)
     (in_bom yes) (on_board yes) (fields_autoplaced)
-    (property "Reference" "#PWR039" (id 0) (at 114.3 45.72 0)
+    (property "Reference" "#PWR?" (id 0) (at 114.3 45.72 0)
       (effects (font (size 1.27 1.27)) hide)
     )
@@
   (symbol (lib_id "power:+3.3V") (at 148.59 35.56 0) (unit 1)
     (in_bom yes) (on_board yes) (fields_autoplaced)
-    (property "Reference" "#PWR041" (id 0) (at 148.59 39.37 0)
-      (effects (font (size 1.27 1.27)) hide)
-    )
+    (property "Reference" "#PWR?" (id 0) (at 148.59 39.37 0)
+      (effects (font (size 1.27 1.27)) hide)
+    )
