File: JetsonCarrierBoard/micro_usb-DESKTOP-4N3HF78.kicad_sch (KiCad schematic)
At the start: 9 parts, among them J8 USB_B_Micro, Q11 DMN24H3D5L

Commit message: A ton
Parts:
- D?: renamed from D31; value D_LES -> LESD5VD8LCG-R
- D?: renamed from D30; value D_LES -> LESD5VD8LCG-R
- renumbered C87 to C?, C86 to C?, D29 to D?, J8 to J?, Q11 to Q?, R78 to R?, R79 to R?
Changed lines of the file:
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@@
   (symbol (lib_id "power:GND") (at 165.1 124.46 0) (unit 1)
     (in_bom yes) (on_board yes) (fields_autoplaced)
-    (property "Reference" "#PWR0195" (id 0) (at 165.1 130.81 0)
+    (property "Reference" "#PWR?" (id 0) (at 165.1 130.81 0)
       (effects (font (size 1.27 1.27)) hide)
     )
@@
   (symbol (lib_id "Transistor_FET:DMN24H3D5L") (at 170.18 83.82 0) (unit 1)
     (in_bom yes) (on_board yes) (fields_autoplaced)
-    (property "Reference" "Q11" (id 0) (at 176.53 82.5499 0)
+    (property "Reference" "Q?" (id 0) (at 176.53 82.5499 0)
       (effects (font (size 1.27 1.27)) (justify left))
     )
@@
   (symbol (lib_id "Device:D_TVS") (at 143.51 120.65 90) (unit 1)
     (in_bom yes) (on_board yes)
-    (property "Reference" "D31" (id 0) (at 146.685 119.38 90)
-      (effects (font (size 1.27 1.27)) (justify right))
-    )
-    (property "Value" "D_LES" (id 1) (at 145.415 121.92 90)
+    (property "Reference" "D?" (id 0) (at 148.59 121.92 90)
+      (effects (font (size 1.27 1.27)) (justify right))
+    )
+    (property "Value" "LESD5VD8LCG-R" (id 1) (at 143.51 124.46 90)
       (effects (font (size 1.27 1.27)) (justify right))
     )
@@
   (symbol (lib_id "Device:D_TVS") (at 111.76 87.63 90) (unit 1)
     (in_bom yes) (on_board yes)
-    (property "Reference" "D29" (id 0) (at 99.06 86.36 90)
+    (property "Reference" "D?" (id 0) (at 99.06 86.36 90)
       (effects (font (size 1.27 1.27)) (justify right))
     )
@@
   (symbol (lib_id "Device:C") (at 133.35 120.65 0) (unit 1)
     (in_bom yes) (on_board yes) (fields_autoplaced)
-    (property "Reference" "C87" (id 0) (at 137.16 119.3799 0)
+    (property "Reference" "C?" (id 0) (at 137.16 119.3799 0)
       (effects (font (size 1.27 1.27)) (justify left))
     )
@@
   (symbol (lib_id "Device:C") (at 129.54 87.63 0) (unit 1)
     (in_bom yes) (on_board yes) (fields_autoplaced)
-    (property "Reference" "C86" (id 0) (at 133.35 86.3599 0)
+    (property "Reference" "C?" (id 0) (at 133.35 86.3599 0)
       (effects (font (size 1.27 1.27)) (justify left))
     )
@@
   (symbol (lib_id "Device:R") (at 144.78 83.82 90) (unit 1)
     (in_bom yes) (on_board yes)
-    (property "Reference" "R78" (id 0) (at 144.78 81.788 90))
+    (property "Reference" "R?" (id 0) (at 144.78 81.788 90))
     (property "Value" "0" (id 1) (at 144.78 83.82 90))
     (property "Footprint" "" (id 2) (at 144.78 85.598 90)
@@
   (symbol (lib_id "power:GND") (at 133.35 127 0) (unit 1)
     (in_bom yes) (on_board yes) (fields_autoplaced)
-    (property "Reference" "#PWR0193" (id 0) (at 133.35 133.35 0)
+    (property "Reference" "#PWR?" (id 0) (at 133.35 133.35 0)
       (effects (font (size 1.27 1.27)) hide)
     )
@@
   (symbol (lib_id "Device:R") (at 157.48 87.63 180) (unit 1)
     (in_bom yes) (on_board yes) (fields_autoplaced)
-    (property "Reference" "R79" (id 0) (at 160.02 86.3599 0)
+    (property "Reference" "R?" (id 0) (at 160.02 86.3599 0)
       (effects (font (size 1.27 1.27)) (justify right))
     )
@@
   (symbol (lib_id "power:GND") (at 129.54 93.98 0) (unit 1)
     (in_bom yes) (on_board yes) (fields_autoplaced)
-    (property "Reference" "#PWR0192" (id 0) (at 129.54 100.33 0)
+    (property "Reference" "#PWR?" (id 0) (at 129.54 100.33 0)
       (effects (font (size 1.27 1.27)) hide)
     )
@@
   (symbol (lib_id "Device:D_TVS") (at 127 120.65 90) (unit 1)
     (in_bom yes) (on_board yes)
-    (property "Reference" "D30" (id 0) (at 120.015 120.015 90)
-      (effects (font (size 1.27 1.27)) (justify right))
-    )
-    (property "Value" "D_LES" (id 1) (at 118.745 122.555 90)
+    (property "Reference" "D?" (id 0) (at 115.57 119.38 90)
+      (effects (font (size 1.27 1.27)) (justify right))
+    )
+    (property "Value" "LESD5VD8LCG-R" (id 1) (at 107.95 121.92 90)
       (effects (font (size 1.27 1.27)) (justify right))
     )
@@
   (symbol (lib_id "Connector:USB_B_Micro") (at 163.83 111.76 0) (mirror y) (unit 1)
     (in_bom yes) (on_board yes) (fields_autoplaced)
-    (property "Reference" "J8" (id 0) (at 170.18 110.4899 0)
+    (property "Reference" "J?" (id 0) (at 170.18 110.4899 0)
       (effects (font (size 1.27 1.27)) (justify right))
     )
@@
   (symbol (lib_id "power:GND") (at 111.76 93.98 0) (unit 1)
     (in_bom yes) (on_board yes) (fields_autoplaced)
-    (property "Reference" "#PWR0190" (id 0) (at 111.76 100.33 0)
+    (property "Reference" "#PWR?" (id 0) (at 111.76 100.33 0)
       (effects (font (size 1.27 1.27)) hide)
     )
@@
   (symbol (lib_id "power:GND") (at 127 127 0) (unit 1)
     (in_bom yes) (on_board yes) (fields_autoplaced)
-    (property "Reference" "#PWR0191" (id 0) (at 127 133.35 0)
+    (property "Reference" "#PWR?" (id 0) (at 127 133.35 0)
       (effects (font (size 1.27 1.27)) hide)
     )
@@
   (symbol (lib_id "power:GND") (at 172.72 93.98 0) (unit 1)
     (in_bom yes) (on_board yes) (fields_autoplaced)
-    (property "Reference" "#PWR0196" (id 0) (at 172.72 100.33 0)
+    (property "Reference" "#PWR?" (id 0) (at 172.72 100.33 0)
       (effects (font (size 1.27 1.27)) hide)
     )
@@
   (symbol (lib_id "power:GND") (at 143.51 127 0) (unit 1)
     (in_bom yes) (on_board yes) (fields_autoplaced)
-    (property "Reference" "#PWR0194" (id 0) (at 143.51 133.35 0)
-      (effects (font (size 1.27 1.27)) hide)
-    )
+    (property "Reference" "#PWR?" (id 0) (at 143.51 133.35 0)
+      (effects (font (size 1.27 1.27)) hide)
+    )
