File: JetsonCarrierBoard/microphone-DESKTOP-4N3HF78.kicad_sch (KiCad schematic)
At the start: 5 parts, among them U8 ICS-43434, U9 ICS-43434

Commit message: A ton
Parts:
- renumbered C55 to C?, C54 to C?, R34 to R?, U8 to U?, U9 to U?
Changed lines of the file:
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@@
   (symbol (lib_id "I2S_MEMS_Microphone:ICS-43434") (at 125.73 105.41 0) (unit 1)
     (in_bom yes) (on_board yes) (fields_autoplaced)
-    (property "Reference" "U8" (id 0) (at 127.7494 92.71 0)
+    (property "Reference" "U?" (id 0) (at 127.7494 92.71 0)
       (effects (font (size 1.27 1.27)) (justify left))
     )
@@
   (symbol (lib_id "power:+1V8") (at 125.73 90.17 0) (unit 1)
     (in_bom yes) (on_board yes) (fields_autoplaced)
-    (property "Reference" "#PWR067" (id 0) (at 125.73 93.98 0)
+    (property "Reference" "#PWR?" (id 0) (at 125.73 93.98 0)
       (effects (font (size 1.27 1.27)) hide)
     )
@@
   (symbol (lib_id "Device:C") (at 177.8 111.76 0) (unit 1)
     (in_bom yes) (on_board yes)
-    (property "Reference" "C55" (id 0) (at 181.61 110.49 0)
+    (property "Reference" "C?" (id 0) (at 181.61 110.49 0)
       (effects (font (size 1.27 1.27)) (justify left))
     )
@@
   (symbol (lib_id "power:+1V8") (at 167.64 90.17 0) (unit 1)
     (in_bom yes) (on_board yes) (fields_autoplaced)
-    (property "Reference" "#PWR069" (id 0) (at 167.64 93.98 0)
+    (property "Reference" "#PWR?" (id 0) (at 167.64 93.98 0)
       (effects (font (size 1.27 1.27)) hide)
     )
@@
   (symbol (lib_id "I2S_MEMS_Microphone:ICS-43434") (at 167.64 105.41 0) (mirror y) (unit 1)
     (in_bom yes) (on_board yes)
-    (property "Reference" "U9" (id 0) (at 162.56 93.98 0))
+    (property "Reference" "U?" (id 0) (at 162.56 93.98 0))
     (property "Value" "ICS-43434" (id 1) (at 158.75 96.5169 0))
     (property "Footprint" "" (id 2) (at 167.64 105.41 0)
@@
   (symbol (lib_id "power:GND") (at 167.64 118.11 0) (unit 1)
     (in_bom yes) (on_board yes) (fields_autoplaced)
-    (property "Reference" "#PWR070" (id 0) (at 167.64 124.46 0)
+    (property "Reference" "#PWR?" (id 0) (at 167.64 124.46 0)
       (effects (font (size 1.27 1.27)) hide)
     )
@@
   (symbol (lib_id "Device:C") (at 115.57 96.52 0) (unit 1)
     (in_bom yes) (on_board yes)
-    (property "Reference" "C54" (id 0) (at 110.49 95.25 0)
+    (property "Reference" "C?" (id 0) (at 110.49 95.25 0)
       (effects (font (size 1.27 1.27)) (justify left))
     )
@@
   (symbol (lib_id "Device:R") (at 146.05 113.03 0) (unit 1)
     (in_bom yes) (on_board yes) (fields_autoplaced)
-    (property "Reference" "R34" (id 0) (at 147.828 112.1953 0)
+    (property "Reference" "R?" (id 0) (at 147.828 112.1953 0)
       (effects (font (size 1.27 1.27)) (justify left))
     )
@@
   (symbol (lib_id "power:GND") (at 125.73 118.11 0) (unit 1)
     (in_bom yes) (on_board yes) (fields_autoplaced)
-    (property "Reference" "#PWR068" (id 0) (at 125.73 124.46 0)
+    (property "Reference" "#PWR?" (id 0) (at 125.73 124.46 0)
       (effects (font (size 1.27 1.27)) hide)
     )
