File: JetsonCarrierBoard/power_mcu-DESKTOP-4N3HF78.kicad_sch (KiCad schematic)
At the start: 36 parts, among them Q8 BSS84, Q9 2N7002, U20 74LVC1G07, U21 EFM8SB10F2G-A-QFN20, U22 SN74LV1T86, U23 SN74LV1T86

Commit message: A ton
Parts:
- renumbered C78 to C?, C79 to C?, C77 to C?, D27 to D?, D26 to D?, Q8 to Q?, Q9 to Q?, R72 to R?, R61 to R?, R64 to R?, R63 to R?, R66 to R?, R69 to R?, R73 to R?, R74 to R?, R58 to R?, R59 to R?, R67 to R?, R70 to R?, R65 to R?, R55 to R?, R75 to R?, R57 to R?, R62 to R?, R68 to R?, R71 to R?, R60 to R?, R56 to R?, TP2 to TP?, TP4 to TP?, TP3 to TP?, TP1 to TP?, U23 to U?, U22 to U?, U20 to U?, U21 to U?
