File: JetsonCarrierBoard/pre-reg3V3-DESKTOP-4N3HF78.kicad_sch (KiCad schematic)
At the start: 22 parts, among them Q1 DMN24H3D5L, Q2 DMN24H3D5L, U3 SIC43x

Commit message: A ton
Parts:
- renumbered C16 to C?, C21 to C?, C18 to C?, C14 to C?, C17 to C?, C15 to C?, C23 to C?, C22 to C?, C20 to C?, C19 to C?, L2 to L?, Q1 to Q?, Q2 to Q?, R23 to R?, R21 to R?, R16 to R?, R20 to R?, R17 to R?, R18 to R?, R19 to R?, R22 to R?, U3 to U?
