File: JetsonCarrierBoard/pre-reg5V-DESKTOP-4N3HF78.kicad_sch (KiCad schematic)
At the start: 20 parts, among them U2 SIC43x

Commit message: A ton
Parts:
- renumbered C8 to C?, C13 to C?, C9 to C?, C11 to C?, C12 to C?, C5 to C?, C10 to C?, C7 to C?, C4 to C?, C6 to C?, L1 to L?, R10 to R?, R13 to R?, R8 to R?, R12 to R?, R14 to R?, R15 to R?, R9 to R?, R11 to R?, U2 to U?
Changed lines of the file:
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@@
   (symbol (lib_id "Voltage_Regulators_Switching:SIC43x") (at 146.05 80.01 0) (unit 1)
     (in_bom yes) (on_board yes) (fields_autoplaced)
-    (property "Reference" "U2" (id 0) (at 146.05 73.66 0))
+    (property "Reference" "U?" (id 0) (at 146.05 73.66 0))
     (property "Value" "SIC43x" (id 1) (at 146.05 76.2 0))
     (property "Footprint" "" (id 2) (at 151.13 80.01 0)
@@
   (symbol (lib_id "Device:C") (at 165.1 78.74 90) (unit 1)
     (in_bom yes) (on_board yes)
-    (property "Reference" "C8" (id 0) (at 167.64 77.47 90))
+    (property "Reference" "C?" (id 0) (at 167.64 77.47 90))
     (property "Value" "1u" (id 1) (at 162.56 77.47 90))
     (property "Footprint" "" (id 2) (at 168.91 77.7748 0)
@@
   (symbol (lib_id "Device:C") (at 201.93 100.33 0) (unit 1)
     (in_bom yes) (on_board yes) (fields_autoplaced)
-    (property "Reference" "C13" (id 0) (at 204.851 99.4953 0)
+    (property "Reference" "C?" (id 0) (at 204.851 99.4953 0)
       (effects (font (size 1.27 1.27)) (justify left))
     )
@@
   (symbol (lib_id "Device:C") (at 165.1 83.82 90) (unit 1)
     (in_bom yes) (on_board yes)
-    (property "Reference" "C9" (id 0) (at 167.64 82.55 90))
+    (property "Reference" "C?" (id 0) (at 167.64 82.55 90))
     (property "Value" "4.7u" (id 1) (at 161.29 82.55 90))
     (property "Footprint" "" (id 2) (at 168.91 82.8548 0)
@@
   (symbol (lib_id "Device:C") (at 181.61 100.33 0) (unit 1)
     (in_bom yes) (on_board yes) (fields_autoplaced)
-    (property "Reference" "C11" (id 0) (at 184.531 99.4953 0)
+    (property "Reference" "C?" (id 0) (at 184.531 99.4953 0)
       (effects (font (size 1.27 1.27)) (justify left))
     )
@@
   (symbol (lib_id "Device:C") (at 191.77 100.33 0) (unit 1)
     (in_bom yes) (on_board yes) (fields_autoplaced)
-    (property "Reference" "C12" (id 0) (at 194.691 99.4953 0)
+    (property "Reference" "C?" (id 0) (at 194.691 99.4953 0)
       (effects (font (size 1.27 1.27)) (justify left))
     )
@@
   (symbol (lib_id "Device:R") (at 127 99.06 90) (unit 1)
     (in_bom yes) (on_board yes)
-    (property "Reference" "R10" (id 0) (at 127 97.028 90))
+    (property "Reference" "R?" (id 0) (at 127 97.028 90))
     (property "Value" "2.2" (id 1) (at 127 99.06 90))
     (property "Footprint" "" (id 2) (at 127 100.838 90)
@@
   (symbol (lib_id "power:GND") (at 130.81 123.19 0) (unit 1)
     (in_bom yes) (on_board yes) (fields_autoplaced)
-    (property "Reference" "#PWR018" (id 0) (at 130.81 129.54 0)
+    (property "Reference" "#PWR?" (id 0) (at 130.81 129.54 0)
       (effects (font (size 1.27 1.27)) hide)
     )
@@
   (symbol (lib_id "power:+BATT") (at 85.09 91.44 0) (unit 1)
     (in_bom yes) (on_board yes) (fields_autoplaced)
-    (property "Reference" "#PWR014" (id 0) (at 85.09 95.25 0)
+    (property "Reference" "#PWR?" (id 0) (at 85.09 95.25 0)
       (effects (font (size 1.27 1.27)) hide)
     )
@@
   (symbol (lib_id "Device:L") (at 165.1 96.52 90) (unit 1)
     (in_bom yes) (on_board yes) (fields_autoplaced)
-    (property "Reference" "L1" (id 0) (at 165.1 92.3122 90))
+    (property "Reference" "L?" (id 0) (at 165.1 92.3122 90))
     (property "Value" "2.2u" (id 1) (at 165.1 94.8491 90))
     (property "Footprint" "" (id 2) (at 165.1 96.52 0)
@@
   (symbol (lib_id "Device:R") (at 165.1 73.66 90) (unit 1)
     (in_bom yes) (on_board yes) (fields_autoplaced)
-    (property "Reference" "R13" (id 0) (at 165.1 68.9442 90))
+    (property "Reference" "R?" (id 0) (at 165.1 68.9442 90))
     (property "Value" "10k" (id 1) (at 165.1 71.4811 90))
     (property "Footprint" "" (id 2) (at 165.1 75.438 90)
@@
   (symbol (lib_id "Device:R") (at 85.09 96.52 0) (unit 1)
     (in_bom yes) (on_board yes) (fields_autoplaced)
-    (property "Reference" "R8" (id 0) (at 86.868 95.6853 0)
+    (property "Reference" "R?" (id 0) (at 86.868 95.6853 0)
       (effects (font (size 1.27 1.27)) (justify left))
     )
@@
   (symbol (lib_id "Device:C") (at 116.84 99.06 90) (unit 1)
     (in_bom yes) (on_board yes) (fields_autoplaced)
-    (property "Reference" "C5" (id 0) (at 116.84 93.2012 90))
+    (property "Reference" "C?" (id 0) (at 116.84 93.2012 90))
     (property "Value" "0.1u" (id 1) (at 116.84 95.7381 90))
     (property "Footprint" "" (id 2) (at 120.65 98.0948 0)
@@
   (symbol (lib_id "Device:C") (at 171.45 100.33 0) (unit 1)
     (in_bom yes) (on_board yes) (fields_autoplaced)
-    (property "Reference" "C10" (id 0) (at 174.371 99.4953 0)
+    (property "Reference" "C?" (id 0) (at 174.371 99.4953 0)
       (effects (font (size 1.27 1.27)) (justify left))
     )
@@
   (symbol (lib_id "power:+5V") (at 201.93 96.52 0) (unit 1)
     (in_bom yes) (on_board yes) (fields_autoplaced)
-    (property "Reference" "#PWR021" (id 0) (at 201.93 100.33 0)
+    (property "Reference" "#PWR?" (id 0) (at 201.93 100.33 0)
       (effects (font (size 1.27 1.27)) hide)
     )
@@
   (symbol (lib_id "Device:R") (at 127 105.41 90) (unit 1)
     (in_bom yes) (on_board yes)
-    (property "Reference" "R12" (id 0) (at 127 107.95 90))
+    (property "Reference" "R?" (id 0) (at 127 107.95 90))
     (property "Value" "200k" (id 1) (at 127 105.41 90))
     (property "Footprint" "" (id 2) (at 127 107.188 90)
@@
   (symbol (lib_id "Device:R") (at 165.1 105.41 90) (unit 1)
     (in_bom yes) (on_board yes)
-    (property "Reference" "R14" (id 0) (at 162.56 102.87 90))
+    (property "Reference" "R?" (id 0) (at 162.56 102.87 90))
     (property "Value" "73k" (id 1) (at 166.37 102.87 90))
     (property "Footprint" "" (id 2) (at 165.1 107.188 90)
@@
   (symbol (lib_id "power:+BATT") (at 130.81 78.74 0) (unit 1)
     (in_bom yes) (on_board yes) (fields_autoplaced)
-    (property "Reference" "#PWR017" (id 0) (at 130.81 82.55 0)
+    (property "Reference" "#PWR?" (id 0) (at 130.81 82.55 0)
       (effects (font (size 1.27 1.27)) hide)
     )
@@
   (symbol (lib_id "power:GND") (at 161.29 123.19 0) (unit 1)
     (in_bom yes) (on_board yes) (fields_autoplaced)
-    (property "Reference" "#PWR019" (id 0) (at 161.29 129.54 0)
+    (property "Reference" "#PWR?" (id 0) (at 161.29 129.54 0)
       (effects (font (size 1.27 1.27)) hide)
     )
@@
   (symbol (lib_id "Device:R") (at 168.91 114.3 0) (unit 1)
     (in_bom yes) (on_board yes) (fields_autoplaced)
-    (property "Reference" "R15" (id 0) (at 171.45 113.0299 0)
+    (property "Reference" "R?" (id 0) (at 171.45 113.0299 0)
       (effects (font (size 1.27 1.27)) (justify left))
     )
@@
   (symbol (lib_id "Device:R") (at 85.09 105.41 0) (unit 1)
     (in_bom yes) (on_board yes) (fields_autoplaced)
-    (property "Reference" "R9" (id 0) (at 86.868 104.5753 0)
+    (property "Reference" "R?" (id 0) (at 86.868 104.5753 0)
       (effects (font (size 1.27 1.27)) (justify left))
     )
@@
   (symbol (lib_id "Device:C") (at 123.19 85.09 0) (unit 1)
     (in_bom yes) (on_board yes) (fields_autoplaced)
-    (property "Reference" "C7" (id 0) (at 126.111 84.2553 0)
+    (property "Reference" "C?" (id 0) (at 126.111 84.2553 0)
       (effects (font (size 1.27 1.27)) (justify left))
     )
@@
   (symbol (lib_id "Device:C") (at 111.76 85.09 0) (unit 1)
     (in_bom yes) (on_board yes) (fields_autoplaced)
-    (property "Reference" "C4" (id 0) (at 114.681 84.2553 0)
+    (property "Reference" "C?" (id 0) (at 114.681 84.2553 0)
       (effects (font (size 1.27 1.27)) (justify left))
     )
@@
   (symbol (lib_id "power:GND") (at 171.45 83.82 0) (unit 1)
     (in_bom yes) (on_board yes)
-    (property "Reference" "#PWR020" (id 0) (at 171.45 90.17 0)
+    (property "Reference" "#PWR?" (id 0) (at 171.45 90.17 0)
       (effects (font (size 1.27 1.27)) hide)
     )
@@
   (symbol (lib_id "Device:C") (at 116.84 120.65 90) (unit 1)
     (in_bom yes) (on_board yes) (fields_autoplaced)
-    (property "Reference" "C6" (id 0) (at 116.84 114.7912 90))
+    (property "Reference" "C?" (id 0) (at 116.84 114.7912 90))
     (property "Value" "100n" (id 1) (at 116.84 117.3281 90))
     (property "Footprint" "" (id 2) (at 120.65 119.6848 0)
@@
   (symbol (lib_id "power:GND") (at 85.09 110.49 0) (unit 1)
     (in_bom yes) (on_board yes) (fields_autoplaced)
-    (property "Reference" "#PWR015" (id 0) (at 85.09 116.84 0)
+    (property "Reference" "#PWR?" (id 0) (at 85.09 116.84 0)
       (effects (font (size 1.27 1.27)) hide)
     )
@@
   (symbol (lib_id "power:GND") (at 120.65 107.95 0) (unit 1)
     (in_bom yes) (on_board yes) (fields_autoplaced)
-    (property "Reference" "#PWR016" (id 0) (at 120.65 114.3 0)
+    (property "Reference" "#PWR?" (id 0) (at 120.65 114.3 0)
       (effects (font (size 1.27 1.27)) hide)
     )
@@
   (symbol (lib_id "Device:R") (at 127 102.87 90) (unit 1)
     (in_bom yes) (on_board yes)
-    (property "Reference" "R11" (id 0) (at 127 101.092 90))
+    (property "Reference" "R?" (id 0) (at 127 101.092 90))
     (property "Value" "499k" (id 1) (at 127 102.87 90))
     (property "Footprint" "" (id 2) (at 127 104.648 90)
