File: JetsonCarrierBoard/sodimm1-DESKTOP-4N3HF78.kicad_sch (KiCad schematic)
At the start: 12 parts, among them J1 CON_SODIMM260_JETSON_NANO

Commit message: A ton
Parts:
- D?: renamed from D2; value D_TPD -> TPD1E10B06
- D?: renamed from D1; value D_TPD -> TPD1E10B06
- renumbered C1 to C?, C2 to C?, C3 to C?, H1 to H?, H2 to H?, J1 to J?, R4 to R?, R3 to R?, R1 to R?, R2 to R?
Changed lines of the file:
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@@
   (symbol (lib_id "Mechanical:MountingHole_Pad") (at 54.61 100.33 0) (unit 1)
     (in_bom yes) (on_board yes) (fields_autoplaced)
-    (property "Reference" "H1" (id 0) (at 57.277 97.7899 0)
+    (property "Reference" "H?" (id 0) (at 57.277 97.7899 0)
       (effects (font (size 1.27 1.27)) (justify left))
     )
@@
   (symbol (lib_id "power:GND") (at 119.38 177.8 0) (unit 1)
     (in_bom yes) (on_board yes)
-    (property "Reference" "#PWR05" (id 0) (at 119.38 184.15 0)
+    (property "Reference" "#PWR?" (id 0) (at 119.38 184.15 0)
       (effects (font (size 1.27 1.27)) hide)
     )
@@
   (symbol (lib_id "Mechanical:MountingHole_Pad") (at 78.105 100.33 0) (unit 1)
     (in_bom yes) (on_board yes) (fields_autoplaced)
-    (property "Reference" "H2" (id 0) (at 80.772 97.7899 0)
+    (property "Reference" "H?" (id 0) (at 80.772 97.7899 0)
       (effects (font (size 1.27 1.27)) (justify left))
     )
@@
   (symbol (lib_id "Device:D_TVS") (at 191.77 120.65 90) (unit 1)
     (in_bom yes) (on_board yes)
-    (property "Reference" "D2" (id 0) (at 196.215 120.015 90)
+    (property "Reference" "D?" (id 0) (at 196.85 122.555 90)
       (effects (font (size 1.27 1.27)) (justify right))
     )
-    (property "Value" "D_TPD" (id 1) (at 194.31 121.92 90)
+    (property "Value" "TPD1E10B06" (id 1) (at 192.405 125.095 90)
       (effects (font (size 1.27 1.27)) (justify right))
     )
@@
   (symbol (lib_id "Device:R") (at 193.04 27.94 0) (unit 1)
     (in_bom yes) (on_board yes) (fields_autoplaced)
-    (property "Reference" "R4" (id 0) (at 195.58 26.6699 0)
+    (property "Reference" "R?" (id 0) (at 195.58 26.6699 0)
       (effects (font (size 1.27 1.27)) (justify left))
     )
@@
   (symbol (lib_id "power:GND") (at 191.77 127 0) (unit 1)
     (in_bom yes) (on_board yes)
-    (property "Reference" "#PWR09" (id 0) (at 191.77 133.35 0)
+    (property "Reference" "#PWR?" (id 0) (at 191.77 133.35 0)
       (effects (font (size 1.27 1.27)) hide)
     )
@@
   (symbol (lib_id "SODIMM_Connector:CON_SODIMM260_JETSON_NANO") (at 144.78 102.87 0) (unit 1)
     (in_bom yes) (on_board yes) (fields_autoplaced)
-    (property "Reference" "J1" (id 0) (at 144.78 24.13 0))
+    (property "Reference" "J?" (id 0) (at 144.78 24.13 0))
     (property "Value" "CON_SODIMM260_JETSON_NANO" (id 1) (at 144.78 26.67 0))
     (property "Footprint" "" (id 2) (at 180.34 59.69 0)
@@
   (symbol (lib_id "power:GND") (at 83.82 43.18 0) (unit 1)
     (in_bom yes) (on_board yes)
-    (property "Reference" "#PWR04" (id 0) (at 83.82 49.53 0)
+    (property "Reference" "#PWR?" (id 0) (at 83.82 49.53 0)
       (effects (font (size 1.27 1.27)) hide)
     )
@@
   (symbol (lib_id "power:GND") (at 177.8 127 0) (unit 1)
     (in_bom yes) (on_board yes)
-    (property "Reference" "#PWR07" (id 0) (at 177.8 133.35 0)
+    (property "Reference" "#PWR?" (id 0) (at 177.8 133.35 0)
       (effects (font (size 1.27 1.27)) hide)
     )
@@
   (symbol (lib_id "Device:C_Polarized") (at 83.82 36.83 0) (unit 1)
     (in_bom yes) (on_board yes) (fields_autoplaced)
-    (property "Reference" "C1" (id 0) (at 86.741 35.1063 0)
+    (property "Reference" "C?" (id 0) (at 86.741 35.1063 0)
       (effects (font (size 1.27 1.27)) (justify left))
     )
@@
   (symbol (lib_id "power:GND") (at 78.105 104.775 0) (unit 1)
     (in_bom yes) (on_board yes)
-    (property "Reference" "#PWR02" (id 0) (at 78.105 111.125 0)
+    (property "Reference" "#PWR?" (id 0) (at 78.105 111.125 0)
       (effects (font (size 1.27 1.27)) hide)
     )
@@
   (symbol (lib_id "power:GND") (at 170.18 177.8 0) (unit 1)
     (in_bom yes) (on_board yes)
-    (property "Reference" "#PWR06" (id 0) (at 170.18 184.15 0)
+    (property "Reference" "#PWR?" (id 0) (at 170.18 184.15 0)
       (effects (font (size 1.27 1.27)) hide)
     )
@@
   (symbol (lib_id "Device:R") (at 185.42 27.94 0) (unit 1)
     (in_bom yes) (on_board yes) (fields_autoplaced)
-    (property "Reference" "R3" (id 0) (at 187.96 26.6699 0)
+    (property "Reference" "R?" (id 0) (at 187.96 26.6699 0)
       (effects (font (size 1.27 1.27)) (justify left))
     )
@@
   (symbol (lib_id "power:GND") (at 54.61 104.775 0) (unit 1)
     (in_bom yes) (on_board yes)
-    (property "Reference" "#PWR01" (id 0) (at 54.61 111.125 0)
+    (property "Reference" "#PWR?" (id 0) (at 54.61 111.125 0)
       (effects (font (size 1.27 1.27)) hide)
     )
@@
   (symbol (lib_id "Device:R") (at 170.18 27.94 0) (unit 1)
     (in_bom yes) (on_board yes) (fields_autoplaced)
-    (property "Reference" "R1" (id 0) (at 172.72 26.6699 0)
+    (property "Reference" "R?" (id 0) (at 172.72 26.6699 0)
       (effects (font (size 1.27 1.27)) (justify left))
     )
@@
   (symbol (lib_id "Device:R") (at 177.8 27.94 0) (unit 1)
     (in_bom yes) (on_board yes) (fields_autoplaced)
-    (property "Reference" "R2" (id 0) (at 180.34 26.6699 0)
+    (property "Reference" "R?" (id 0) (at 180.34 26.6699 0)
       (effects (font (size 1.27 1.27)) (justify left))
     )
@@
   (symbol (lib_id "Device:C_Polarized") (at 96.52 36.83 0) (unit 1)
     (in_bom yes) (on_board yes) (fields_autoplaced)
-    (property "Reference" "C2" (id 0) (at 99.441 35.1063 0)
+    (property "Reference" "C?" (id 0) (at 99.441 35.1063 0)
       (effects (font (size 1.27 1.27)) (justify left))
     )
@@
   (symbol (lib_id "power:+3.3V") (at 181.61 21.59 0) (unit 1)
     (in_bom yes) (on_board yes) (fields_autoplaced)
-    (property "Reference" "#PWR08" (id 0) (at 181.61 25.4 0)
+    (property "Reference" "#PWR?" (id 0) (at 181.61 25.4 0)
       (effects (font (size 1.27 1.27)) hide)
     )
@@
   (symbol (lib_id "Device:D_TVS") (at 177.8 120.65 90) (unit 1)
     (in_bom yes) (on_board yes)
-    (property "Reference" "D1" (id 0) (at 182.245 120.015 90)
+    (property "Reference" "D?" (id 0) (at 182.88 122.555 90)
       (effects (font (size 1.27 1.27)) (justify right))
     )
-    (property "Value" "D_TPD" (id 1) (at 180.34 121.92 90)
+    (property "Value" "TPD1E10B06" (id 1) (at 178.435 125.095 90)
       (effects (font (size 1.27 1.27)) (justify right))
     )
@@
   (symbol (lib_id "power:+5V") (at 83.82 30.48 0) (unit 1)
     (in_bom yes) (on_board yes) (fields_autoplaced)
-    (property "Reference" "#PWR03" (id 0) (at 83.82 34.29 0)
+    (property "Reference" "#PWR?" (id 0) (at 83.82 34.29 0)
       (effects (font (size 1.27 1.27)) hide)
     )
@@
   (symbol (lib_id "Device:C_Polarized") (at 109.22 36.83 0) (unit 1)
     (in_bom yes) (on_board yes) (fields_autoplaced)
-    (property "Reference" "C3" (id 0) (at 112.141 35.1063 0)
-      (effects (font (size 1.27 1.27)) (justify left))
-    )
+    (property "Reference" "C?" (id 0) (at 112.141 35.1063 0)
+      (effects (font (size 1.27 1.27)) (justify left))
+    )
