File: JetsonCarrierBoard/sodimm2-DESKTOP-4N3HF78.kicad_sch (KiCad schematic)
At the start: 3 parts, among them J1 CON_SODIMM260_JETSON_NANO, U1 74LVC1G07

Commit message: A ton
Parts:
- removed J1: CON_SODIMM260_JETSON_NANO, symbol SODIMM_Connector:CON_SODIMM260_JETSON_NANO
- removed R7: 10k, symbol Device:R
- removed U1: 74LVC1G07, symbol 74xGxx:74LVC1G07
- added J?: CON_SODIMM260_JETSON_NANO, symbol SODIMM_Connector:CON_SODIMM260_JETSON_NANO
- added R? (x2): 1.6k, symbol Device:R
Connections:
- net +3.3V: now also R?.1, R?.1
- new net BT_M2_EN: J?.126 (GPIO03)
- new net CAM0_MCLK: J?.116 (CAM0_MCLK)
- new net CAM0_PWDN: J?.114 (CAM0_PWDN)
- new net CAM1_MCLK: J?.122 (CAM1_MCLK)
- new net CAM1_PWDN: J?.120 (CAM1_PWDN)
- new net CAM_I2C_SCL: J?.213 (CAM_I2C_SCL), R?.2
- new net CAM_I2C_SDA: J?.215 (CAM_I2C_SDA), R?.2
- new net CAM_MUX_SEL: J?.130 (GPIO06)
- new net CSI0_CLK_N: J?.10 (~{CSI0_CLK})
- new net CSI0_CLK_P: J?.12 (CSI0_CLK)
- new net CSI0_D0_N: J?.4 (~{CSI0_D0})
- new net CSI0_D0_P: J?.6 (CSI0_D0)
- new net CSI0_D1_N: J?.16 (~{CSI0_D1})
- new net CSI0_D1_P: J?.18 (CSI0_D1)
- new net CSI2_CLK_N: J?.28 (~{CSI2_CLK})
- new net CSI2_CLK_P: J?.30 (CSI2_CLK)
- new net CSI2_D0_N: J?.22 (~{CSI2_D0})
- new net CSI2_D0_P: J?.24 (CSI2_D0)
- new net CSI2_D1_N: J?.34 (~{CSI2_D1})
- new net CSI2_D1_P: J?.36 (CSI2_D1)
- new net FAN_PWM: J?.230 (GPIO14(PWM))
- new net FAN_TACH: J?.208 (GPIO08(SDMMC_CD))
- new net GPIO01: J?.118 (GPIO01(CLK))
- new net GPIO02: J?.124 (GPIO02)
- new net GPIO07: J?.206 (GPIO07(PWM))
- new net GPIO09: J?.211 (GPIO09(AUD_MCLK))
- new net GPIO10: J?.212 (GPIO10)
- new net GPIO11: J?.216 (GPIO11(CLK))
- new net GPIO12: J?.218 (GPIO12)
- new net GPIO13: J?.228 (GPIO13(PWM))
- new net I2S1_LRCK: J?.224 (I2S1_FS)
- new net I2S1_SCLK: J?.226 (I2S1_SCLK)
- new net I2S1_SDIN: J?.222 (I2S1_DIN)
- new net I2S1_SDOUT: J?.220 (I2S1_DOUT)
- new net MIC_SCK: J?.199 (I2S0_SCLK)
- new net MIC_SD: J?.195 (I2S0_DIN)
- new net MIC_WS: J?.197 (I2S0_FS)
- new net PWR_LED_CTRL: J?.127 (GPIO04)
- new net SPI0_CS0: J?.95 (~{SPI0_CS0})
- new net SPI0_MISO: J?.93 (SPI0_MISO)
- new net SPI0_MOSI: J?.89 (SPI0_MOSI)
- new net SPI0_SCK: J?.91 (SPI0_SCK)
- new net SPI1_CS0: J?.110 (~{SPI1_CS0})
- new net SPI1_MISO: J?.108 (SPI1_MISO)
- new net SPI1_MOSI: J?.104 (SPI1_MOSI)
- new net SPI1_SCK: J?.106 (SPI1_SCK)
- new net USB0_VBUS_DET*: J?.87 (GPIO00(USB_VBUS_EN0))
- new net USB_AP_N: J?.121 (~{USB2_D})
- new net USB_AP_P: J?.123 (USB2_D)
- new net USB_C_DN: J?.115 (~{USB1_D})
- new net USB_C_DP: J?.117 (USB1_D)
- new net USB_M_DN: J?.109 (~{USB0_D})
- new net USB_M_DP: J?.111 (USB0_D)
- new net W_DISABLE1_CTRL: J?.128 (GPIO05)
- no-connect marks 18 -> 41
Other:
- note added: "CAM FPC Con"
- note added: "CAM FPC Con Multiplexed"
- note added: "IMU"
- note added: "M.2 BT"
- note added: "Stereo Microphone"
- note added: "USB Type-C Con"
- note added: "uUSB Con"
- note removed: "DP Con"
- note removed: "M.2 Key E WiFi/BT"
- note removed: "NVME SSD"
- note removed: "USB Type-C Con (USBSS)"
- title: SODIMM Connector 3/3 -> SODIMM Connector 2/3
