File: JetsonCarrierBoard/sodimm3-DESKTOP-4N3HF78.kicad_sch (KiCad schematic)
At the start: 3 parts, among them J1 CON_SODIMM260_JETSON_NANO, U1 74LVC1G07

Commit message: A ton
Parts:
- renumbered J1 to J?, R7 to R?, U1 to U?
Changed lines of the file:
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@@
   (symbol (lib_id "SODIMM_Connector:CON_SODIMM260_JETSON_NANO") (at 130.81 97.79 0) (unit 3)
     (in_bom yes) (on_board yes) (fields_autoplaced)
-    (property "Reference" "J1" (id 0) (at 130.81 39.37 0))
+    (property "Reference" "J?" (id 0) (at 130.81 39.37 0))
     (property "Value" "CON_SODIMM260_JETSON_NANO" (id 1) (at 130.81 41.91 0))
     (property "Footprint" "" (id 2) (at 166.37 54.61 0)
@@
   (symbol (lib_id "power:+3.3V") (at 93.98 154.94 0) (unit 1)
     (in_bom yes) (on_board yes) (fields_autoplaced)
-    (property "Reference" "#PWR013" (id 0) (at 93.98 158.75 0)
+    (property "Reference" "#PWR?" (id 0) (at 93.98 158.75 0)
       (effects (font (size 1.27 1.27)) hide)
     )
@@
   (symbol (lib_id "74xGxx:74LVC1G07") (at 82.55 165.1 0) (unit 1)
     (in_bom yes) (on_board yes)
-    (property "Reference" "U1" (id 0) (at 76.2 157.48 0))
+    (property "Reference" "U?" (id 0) (at 76.2 157.48 0))
     (property "Value" "74LVC1G07" (id 1) (at 76.2 160.02 0))
     (property "Footprint" "" (id 2) (at 82.55 165.1 0)
@@
   (symbol (lib_id "Device:R") (at 93.98 161.29 0) (unit 1)
     (in_bom yes) (on_board yes) (fields_autoplaced)
-    (property "Reference" "R7" (id 0) (at 96.52 160.0199 0)
+    (property "Reference" "R?" (id 0) (at 96.52 160.0199 0)
       (effects (font (size 1.27 1.27)) (justify left))
     )
@@
   (symbol (lib_id "power:+1V8") (at 82.55 158.75 0) (unit 1)
     (in_bom yes) (on_board yes) (fields_autoplaced)
-    (property "Reference" "#PWR011" (id 0) (at 82.55 162.56 0)
+    (property "Reference" "#PWR?" (id 0) (at 82.55 162.56 0)
       (effects (font (size 1.27 1.27)) hide)
     )
@@
   (symbol (lib_id "power:GND") (at 82.55 170.18 0) (unit 1)
     (in_bom yes) (on_board yes) (fields_autoplaced)
-    (property "Reference" "#PWR012" (id 0) (at 82.55 176.53 0)
-      (effects (font (size 1.27 1.27)) hide)
-    )
+    (property "Reference" "#PWR?" (id 0) (at 82.55 176.53 0)
+      (effects (font (size 1.27 1.27)) hide)
+    )
