File: JetsonCarrierBoard/usbC-DESKTOP-4N3HF78.kicad_sch (KiCad schematic)
At the start: 27 parts, among them J4 USB_C_Receptacle, U5 TPS65987D, U6 TPD6S300A, U7 HD3SS460

Commit message: A ton
Parts:
- removed C?: 10u, symbol Device:C
- removed R? (x2): 10k, symbol Device:R
- removed R?: (no value), symbol Device:R
- C?: renamed from C42; value (none) -> 10u
- renumbered C41 to C?, C52 to C?, C46 to C?, C43 to C?, C51 to C?, C45 to C?, C50 to C?, C44 to C?, C48 to C?, C47 to C?, C53 to C?, C49 to C?, D3 to D?, J4 to J?, R29 to R?, R31 to R?, R33 to R?, R32 to R?, R30 to R?, U5 to U?, U6 to U?, U7 to U?
Connections:
- net ADCIN1 is gone; now on net GND: U?.6 (ADCIN1)
- net GND: now also U?.10 (ADCIN2); no longer U?.11 (PP_HV1), U?.12 (PP_HV1), U?.44 (HRESET)
- new net +20V: U?.11 (PP_HV1), U?.12 (PP_HV1)
